File: BluePill.kicad_pcb (KiCad board)
At the start: 2 copper layers, 40.2 x 59.9 mm, 75 parts, among them J1 SWD, J3 Conn_02x08_Odd_Even, J4 BM04B-SURS-TFLFSN, J5 Conn_02x04_Odd_Even, J6 Conn_02x04_Odd_Even, J7 Conn_01x05, J8 Conn_01x04, J9 2169900003, Q1 AO3401A, SW1 SW_SPDT, U1 LM2842X, U2 STM32F405RGT6, U3 USBLC6-2SC6, U4 ICM-42670-P, U5 SN65HVD232QDRQ1, Y1 16MHz

Commit message: siobgg:
Parts:
- removed J8: Conn_01x04, Connector_PinHeader_2.54mm:PinHeader_1x04_P2.54mm_Vertical
- added IC1: ADP2301AUJZ-R7, SnapEDA Library:SOT95P280X100-6N, F.Cu at (125.4, 55.4)
- added IC2: ADP2301AUJZ-R7, SnapEDA Library:SOT95P280X100-6N, F.Cu at (125.3, 86.9)
- added J2: TE 338069-4, SnapEDA Library:TE_338069-4, F.Cu at (66.3, 50.3)
- added U6: XT30PW-F, Connector_AMASS:AMASS_XT30PW-F_1x02_P2.50mm_Horizontal, F.Cu at (119.9, 73.5)
- added U7: XT30PW-M, Connector_AMASS:AMASS_XT30PW-M_1x02_P2.50mm_Horizontal, F.Cu at (131.6, 73.5)
- J9: footprint USB C:MOLEX_2169900003 -> SnapEDA Library:MOLEX_2169900003
Connections:
- J9 pad A6: CONN_USB_D+ -> unconnected-(J9-PadA6)
- J9 pad A7: CONN_USB_D- -> unconnected-(J9-PadA7)
Routing:
- net /Power/COMMON_GND: track 0.00 -> 39.4 mm, vias 0 -> 2
- net unconnected-(J9-PadS1): track 22.2 -> 0.00 mm
- net /Power/V_SUPPLY: track 0.00 -> 20.8 mm
- net /Microcontroller/MCU_BOOT1: track 9.92 -> 9.37 mm
- added copper zone on B.Cu, net /Power/COMMON_GND
- added copper zone on F.Cu, net /Power/V_SUPPLY
Other:
- board size 40.2 x 59.9 mm -> 95.2 x 73.2 mm

Commit message: adsigjningh
Parts:
- added C21: 10u, Capacitor_SMD:C_0402_1005Metric, F.Cu at (126.8, 86.3)
- added C22: 10u 25V, Capacitor_SMD:C_0402_1005Metric, F.Cu at (125.3, 89.1)
- added C23: C1005X5R1E104K050BC, SnapEDA Library:CAPC1005X55N, F.Cu at (122.6, 84.4)
- added C24: 0.1u, Capacitor_SMD:C_0402_1005Metric, F.Cu at (123.3, 90.2)
- added D13: D_Schottky, SnapEDA Library:B230A-13-F, F.Cu at (129.0, 82.0)
- added J8: Conn_01x02, SnapEDA Library:JST_BM02B-SURS-TF(LF)(SN), F.Cu at (118.1, 87.5)
- added L2: 4.7u 2.0A, SnapEDA Library:CDRH5D28RHPNP-4R7NC, F.Cu at (132.5, 90.3)
- added R19: 56k, Resistor_SMD:R_0402_1005Metric, F.Cu at (128.1, 87.4)
- added R20: 10.2k, Resistor_SMD:R_0402_1005Metric, F.Cu at (126.9, 88.5)
- added R21: 31.6k, Resistor_SMD:R_0402_1005Metric, F.Cu at (121.7, 89.7)
- added R22: 10.2k, Resistor_SMD:R_0402_1005Metric, F.Cu at (123.3, 89.1)
- added U8: LSF0102DCUR, SnapEDA Library:SOP50P310X90-8N, F.Cu at (44.7, 76.6)
- J4: footprint BM04B:BM04B-SURS-TFLFSN -> SnapEDA Library:JST_BM04B-SURS-TF(LF)(SN)
- moved U7 3.30 mm to (128.3, 73.6)
- moved IC2 1.24 mm to (124.0, 86.8)
- moved IC1 0.88 mm to (124.5, 55.3), turned to 0 degrees
Connections:
- net /Power/COMMON_GND renamed Earth
- net /Power/V_SUPPLY renamed VS
- IC2 pad 1: unconnected-(IC2-Pad1) -> Net-(IC2-Pad1)
- IC2 pad 3: unconnected-(IC2-Pad3) -> Net-(IC2-Pad3)
- IC2 pad 4: unconnected-(IC2-Pad4) -> Net-(IC2-Pad4)
- IC2 pad 6: unconnected-(IC2-Pad6) -> Net-(D13-Pad1)
Routing:
- net Earth: track 39.4 -> 10.1 mm, vias 2 -> 4
- net +3V3: track 209.9 -> 233.9 mm, vias 6 -> 7
- net MCU_I2C1_SCL: track 22.5 -> 0.00 mm
- net VS: track 20.8 -> 35.5 mm
- net Net-(D13-Pad1): track 0.00 -> 5.82 mm, vias 0 -> 2
- net Net-(IC2-Pad4): track 0.00 -> 2.92 mm
- net Net-(IC2-Pad3): track 0.00 -> 2.41 mm
- net Net-(IC2-Pad1): track 0.00 -> 1.70 mm
- net Net-(J4-Pad4): track 1.55 -> 0.00 mm, vias 1 -> 0
- net Net-(C24-Pad2): track 0.00 -> 1.09 mm
Other:
- board size 95.2 x 73.2 mm -> 91.9 x 73.2 mm

Commit message: skgnigniogni
Parts:
- removed R11, R9: 2k2, Resistor_SMD:R_0402_1005Metric
- added C25: C0603C105K3RACTU, SnapEDA Library:C0603C105K3RACTU, F.Cu at (44.5, 24.2)
- added C26: C0603C105K3RACTU, SnapEDA Library:C0603C105K3RACTU, F.Cu at (48.6, 21.2)
- added U9: LP5907QMFX-3.3Q1, SnapEDA Library:SOT95P280X145-5N, F.Cu at (45.4, 21.4)
- moved L2 170.9 mm to (-9.13, -5.24)
- moved R20 169.1 mm to (-15.0, -3.50)
- moved C21 169.1 mm to (-15.1, -5.61)
- moved C22 169.1 mm to (-16.6, -2.81)
- moved C23 169.1 mm to (-19.3, -7.52)
- moved C24 169.1 mm to (-18.6, -1.75)
- moved IC2 169.1 mm to (-17.9, -5.12)
- moved J8 169.1 mm to (-23.8, -4.46)
- moved R19 169.1 mm to (-13.8, -4.58)
- moved R21 169.1 mm to (-20.2, -2.30)
- moved R22 169.1 mm to (-18.6, -2.81)
- moved U6 169.1 mm to (-21.9, -18.4)
- moved U7 169.1 mm to (-13.6, -18.4)
- moved D13 169.1 mm to (-12.1, -11.2), turned to 180 degrees
- moved IC1 166.4 mm to (-17.4, -31.6)
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Connections:
- U8 pad 1: unconnected-(U8-Pad1) -> GND
- U8 pad 2: unconnected-(U8-Pad2) -> +5V
- U8 pad 3: unconnected-(U8-Pad3) -> Servo_RXD
- U8 pad 4: unconnected-(U8-Pad4) -> Servo_TXD
- U8 pad 5: unconnected-(U8-Pad5) -> MCU_TXD
- U8 pad 6: unconnected-(U8-Pad6) -> MCU_RXD
- U8 pad 7: unconnected-(U8-Pad7) -> +3V3
Routing:
- net +3V3: track 233.9 -> 211.4 mm
- net MCU_I2C1_SCL: track 0.00 -> 22.5 mm
Other:
- board size 91.9 x 73.2 mm -> 75 x 100 mm

Commit message: sgsegwaebdd
Parts:
- removed J8: Conn_01x02, SnapEDA Library:JST_BM02B-SURS-TF(LF)(SN)
- added R11: 2k2, Resistor_SMD:R_0402_1005Metric, F.Cu at (4.99, 34.0)
- added R9: 2k2, Resistor_SMD:R_0402_1005Metric, F.Cu at (4.99, 37.0)
- moved L2 3.89 mm to (-6.86, -8.40), turned to 0 degrees
- moved R17 2.53 mm to (-12.6, 37.6)
- moved J4 2.53 mm to (-10.2, 33.8)
- moved JP1 2.53 mm to (-3.52, 37.3)
- moved JP2 2.53 mm to (-3.52, 33.5)
- moved R18 2.53 mm to (-9.73, 37.6)
- moved D13 1.14 mm to (-12.6, -10.2), turned to 90 degrees
Routing:
- net VS: track 35.1 -> 45.5 mm

Commit message: sdgionbidnb
Parts:
- added R23: 56, Resistor_SMD:R_0402_1005Metric, F.Cu at (-22.4, -34.5)
- added R24: 6.8, Resistor_SMD:R_0402_1005Metric, F.Cu at (-26.1, -31.8)
- added R25: 56k, Resistor_SMD:R_0402_1005Metric, F.Cu at (-25.3, -34.5)
- added R26: 10.2k, Resistor_SMD:R_0402_1005Metric, F.Cu at (-23.2, -31.8)
- C23: value C1005X5R1E104K050BC -> 0.1u ceramic X5R
- IC1, IC2: footprint SnapEDA Library:SOT95P280X100-6N -> BM04B:SOT95P280X100-6N
- J9: footprint SnapEDA Library:MOLEX_2169900003 -> BM04B:MOLEX_2169900003
- R21: value 31.6k -> 52.3
- R22: value 10.2k -> 10
- moved R22 5.18 mm to (-21.8, -6.89)
- moved R20 5.18 mm to (-18.1, -7.58)
- moved IC2 5.18 mm to (-21.1, -9.20)
- moved C21 5.18 mm to (-18.2, -9.69)
- moved C22 5.18 mm to (-19.8, -6.89)
- moved C23 5.18 mm to (-22.5, -11.6)
- moved C24 5.18 mm to (-21.8, -5.83)
- moved R19 5.18 mm to (-17.0, -8.66)
- moved R21 5.18 mm to (-23.3, -6.38)
- moved D13 1.36 mm to (-13.9, -10.2)
- moved L2 1.02 mm to (-7.85, -8.65)
Connections:
- IC1 pad 1: unconnected-(IC1-Pad1) -> Net-(IC1-Pad1)
- IC1 pad 3: unconnected-(IC1-Pad3) -> Net-(IC1-Pad3)
- IC1 pad 4: unconnected-(IC1-Pad4) -> Net-(IC1-Pad4)
- IC1 pad 6: unconnected-(IC1-Pad6) -> Net-(IC1-Pad6)
- L2 pad 2: Net-(C24-Pad2) -> +5V
- R21 pad 1: Net-(C24-Pad2) -> +5V
- U8 pad 2: +5V -> +3V3
- U8 pad 7: +3V3 -> +5V
Routing:
- net +5V: track 5.05 -> 24.9 mm
- net Net-(C23-Pad2): track 5.82 -> 16.1 mm
- net Earth: track 10.1 -> 12.1 mm, vias 4 -> 5
- net VS: track 45.5 -> 44.4 mm
- net Net-(C24-Pad2): track 1.09 -> 0.00 mm

Commit message: WEBGIOWEBGIOBWEG
Parts:
- removed C1, C7, C9: 2u2, Capacitor_SMD:C_0603_1608Metric
- removed C10, C11, C12, C13, C14, C15, C17, C19, C2, C20, C8: 100n, Capacitor_SMD:C_0402_1005Metric
- removed C16: 10n, Capacitor_SMD:C_0402_1005Metric
- removed C18: 2u2, Capacitor_SMD:C_0402_1005Metric
- removed C21: 10u, Capacitor_SMD:C_0402_1005Metric
- removed C22: 10u 25V, Capacitor_SMD:C_0402_1005Metric
- removed C23: 0.1u ceramic X5R, SnapEDA Library:CAPC1005X55N
- removed C24: 0.1u, Capacitor_SMD:C_0402_1005Metric
- removed C25, C26: C0603C105K3RACTU, SnapEDA Library:C0603C105K3RACTU
- removed C3, C6: 10u, Capacitor_SMD:C_0603_1608Metric
- removed C4, C5: 10p, Capacitor_SMD:C_0402_1005Metric
- removed D1: LM5Z2V7T1G, Diode_SMD:D_SOD-523
- removed D10, D11, D12, D5, D6, D7, D8, D9: RCLAMP0521P-N, Diode_SMD:D_0402_1005Metric
- removed D13: D_Schottky, SnapEDA Library:B230A-13-F
- removed D2: B5819W, Diode_SMD:D_SOD-123
- removed D3: GREEN, LED_SMD:LED_0603_1608Metric
- removed D4: BLUE, LED_SMD:LED_0603_1608Metric
- removed FB1, FB2: 100R, Inductor_SMD:L_0603_1608Metric
- removed H1, H2, H3, H4: MountingHole_Pad, MountingHole:MountingHole_3.2mm_M3_Pad_Via
- removed IC1, IC2: ADP2301AUJZ-R7, BM04B:SOT95P280X100-6N
- removed J1: SWD, Connector_PinHeader_1.27mm:PinHeader_2x05_P1.27mm_Vertical
- removed J2: TE 338069-4, SnapEDA Library:TE_338069-4
- removed J3: Conn_02x08_Odd_Even, Connector_PinHeader_2.54mm:PinHeader_2x08_P2.54mm_Vertical
- removed J4: BM04B-SURS-TFLFSN, SnapEDA Library:JST_BM04B-SURS-TF(LF)(SN)
- removed J5, J6: Conn_02x04_Odd_Even, Connector_PinHeader_2.54mm:PinHeader_2x04_P2.54mm_Vertical
- removed J7: Conn_01x05, Connector_PinSocket_2.54mm:PinSocket_1x05_P2.54mm_Vertical
- removed J9: 2169900003, BM04B:MOLEX_2169900003
- removed JP1, JP2: SolderJumper_3_Bridged12, Jumper:SolderJumper-3_P1.3mm_Bridged12_Pad1.0x1.5mm
- removed L1: 15u, BluePhil-Footprints:MPIT4018-150M-LF
- removed L2: 4.7u 2.0A, SnapEDA Library:CDRH5D28RHPNP-4R7NC
- removed Q1: AO3401A, Package_TO_SOT_SMD:SOT-23
- removed R1: 470R, Resistor_SMD:R_0402_1005Metric
- removed R10, R11, R12, R9: 2k2, Resistor_SMD:R_0402_1005Metric
- removed R13, R14, R15: 22R, Resistor_SMD:R_0402_1005Metric
- removed R16: 120R, Resistor_SMD:R_0402_1005Metric
- removed R17, R18, R5: 0R, Resistor_SMD:R_0402_1005Metric
- removed R19, R25: 56k, Resistor_SMD:R_0402_1005Metric
- removed R2: 1k02, Resistor_SMD:R_0402_1005Metric
- removed R20, R26: 10.2k, Resistor_SMD:R_0402_1005Metric
- removed R21: 52.3, Resistor_SMD:R_0402_1005Metric
- removed R22: 10, Resistor_SMD:R_0402_1005Metric
- removed R23: 56, Resistor_SMD:R_0402_1005Metric
- removed R24: 6.8, Resistor_SMD:R_0402_1005Metric
- removed R3: 3k4, Resistor_SMD:R_0402_1005Metric
- removed R4, R7: 1k, Resistor_SMD:R_0402_1005Metric
- removed R6, R8: 10k, Resistor_SMD:R_0402_1005Metric
- removed SW1: SW_SPDT, Button_Switch_SMD:SW_SPDT_PCM12
- removed U1: LM2842X, Package_TO_SOT_SMD:TSOT-23-6
- removed U2: STM32F405RGT6, Package_QFP:LQFP-64_10x10mm_P0.5mm
- removed U3: USBLC6-2SC6, Package_TO_SOT_SMD:SOT-23-6
- removed U4: ICM-42670-P, SnapEDA Library:IC_ICM-42670-P
- removed U5: SN65HVD232QDRQ1, SnapEDA Library:SOIC127P599X175-8N
- removed U6: XT30PW-F, Connector_AMASS:AMASS_XT30PW-F_1x02_P2.50mm_Horizontal
- removed U7: XT30PW-M, Connector_AMASS:AMASS_XT30PW-M_1x02_P2.50mm_Horizontal
- removed U8: LSF0102DCUR, SnapEDA Library:SOP50P310X90-8N
- removed U9: LP5907QMFX-3.3Q1, SnapEDA Library:SOT95P280X145-5N
- removed Y1: 16MHz, Crystal:Crystal_SMD_3225-4Pin_3.2x2.5mm
- added C201: 1u ceramic X7R, SnapEDA Library:C0603C105K3RACTU, F.Cu at (-7.30, -72.0)
- added C202: 0.1u ceramic X5R, SnapEDA Library:CAPC1005X55N, F.Cu at (-46.1, -47.7)
- added C203: 2u2, Capacitor_SMD:C_0603_1608Metric, F.Cu at (-15.7, -64.2)
- added C204: 10u ceramic X5R, SnapEDA Library:CAPC1608X90N, F.Cu at (-15.7, -61.7)
- added C205: 1u ceramic X7R, SnapEDA Library:C0603C105K3RACTU, F.Cu at (-12.4, -67.5)
- added C206: 100n, Capacitor_SMD:C_0402_1005Metric, F.Cu at (-17.1, -59.5)
- added C207: 10u ceramic X5R, SnapEDA Library:CAPC1608X90N, F.Cu at (-21.9, -55.1)
- added C208: 10u, Capacitor_SMD:C_0603_1608Metric, F.Cu at (-20.6, -59.8)
- added C209: 0.1u ceramic X5R, SnapEDA Library:CAPC1005X55N, F.Cu at (-46.1, -49.9)
- added C210: 10u ceramic X5R, SnapEDA Library:CAPC1608X90N, F.Cu at (-29.1, -48.1)
- added C211: 10u ceramic X5R, SnapEDA Library:CAPC1608X90N, F.Cu at (-34.3, -46.2)
- added C301: 10p, Capacitor_SMD:C_0402_1005Metric, F.Cu at (89.7, 42.9)
- added C302: 10p, Capacitor_SMD:C_0402_1005Metric, F.Cu at (105.9, 27.0)
- added C303: 10u, Capacitor_SMD:C_0603_1608Metric, F.Cu at (77.2, 42.0)
- added C304: 2u2, Capacitor_SMD:C_0603_1608Metric, F.Cu at (72.0, 43.9)
- added C305: 100n, Capacitor_SMD:C_0402_1005Metric, F.Cu at (105.9, 29.0)
- added C306: 2u2, Capacitor_SMD:C_0603_1608Metric, F.Cu at (77.2, 39.5)
- added C307: 100n, Capacitor_SMD:C_0402_1005Metric, F.Cu at (92.8, 40.9)
- added C308: 100n, Capacitor_SMD:C_0402_1005Metric, F.Cu at (109.1, 24.4)
- added C309: 100n, Capacitor_SMD:C_0402_1005Metric, F.Cu at (95.8, 38.9)
- added C310: 100n, Capacitor_SMD:C_0402_1005Metric, F.Cu at (108.8, 27.0)
- added C311: 100n, Capacitor_SMD:C_0402_1005Metric, F.Cu at (95.8, 36.9)
- added C312: 100n, Capacitor_SMD:C_0402_1005Metric, F.Cu at (103.0, 31.0)
- added C401: 10n, Capacitor_SMD:C_0402_1005Metric, F.Cu at (49.0, 75.6)
- added C402: 0.1u, Capacitor_SMD:C_0402_1005Metric, F.Cu at (49.9, 69.3)
- added C403: 2u2, Capacitor_SMD:C_0402_1005Metric, F.Cu at (49.9, 71.2)
- added C501: 100n, Capacitor_SMD:C_0402_1005Metric, F.Cu at (19.4, -25.3)
- added C502: 100n, Capacitor_SMD:C_0402_1005Metric, F.Cu at (15.7, -23.6)
- added C503: 100n, Capacitor_SMD:C_0402_1005Metric, F.Cu at (-42.0, -4.89)
- added C504: 100n, Capacitor_SMD:C_0402_1005Metric, F.Cu at (-44.9, -4.89)
- added D201: LM5Z2V7T1G, Diode_SMD:D_SOD-523, F.Cu at (-8.68, -67.6)
- added D202: 30V 2A, SnapEDA Library:B230A-13-F, F.Cu at (-32.8, -54.1)
- added D203: B5819W, Diode_SMD:D_SOD-123, F.Cu at (-41.6, -53.7)
- added D204: GREEN, LED_SMD:LED_0603_1608Metric, F.Cu at (-51.2, -45.2)
- added D205: GREEN, LED_SMD:LED_0603_1608Metric, F.Cu at (-47.2, -45.2)
- added D206: 30V 2A, SnapEDA Library:B230A-13-F, F.Cu at (-48.2, -53.2)
- added D301: BLUE, LED_SMD:LED_0603_1608Metric, F.Cu at (103.6, 22.7)
- added D302: RCLAMP0521P-N, Diode_SMD:D_0402_1005Metric, F.Cu at (87.1, 36.9)
- added D303: RCLAMP0521P-N, Diode_SMD:D_0402_1005Metric, F.Cu at (87.1, 38.9)
- added D304: RCLAMP0521P-N, Diode_SMD:D_0402_1005Metric, F.Cu at (75.7, 44.2)
- added D305: RCLAMP0521P-N, Diode_SMD:D_0402_1005Metric, F.Cu at (103.3, 25.0)
- added D306: RCLAMP0521P-N, Diode_SMD:D_0402_1005Metric, F.Cu at (73.7, 18.2)
- added D501: RCLAMP0521P-N, Diode_SMD:D_0402_1005Metric, F.Cu at (15.8, -28.3)
- added D502: RCLAMP0521P-N, Diode_SMD:D_0402_1005Metric, F.Cu at (18.4, -31.5)
- added D503: RCLAMP0521P-N, Diode_SMD:D_0402_1005Metric, F.Cu at (22.9, -36.2)
- added FB201: 100R, Inductor_SMD:L_0603_1608Metric, F.Cu at (-27.1, -50.6)
- added FB501: 100R, Inductor_SMD:L_0603_1608Metric, F.Cu at (19.2, -35.9)
- added H501: MountingHole_Pad, MountingHole:MountingHole_3.2mm_M3_Pad_Via, F.Cu at (56.7, 37.2)
- added H502: MountingHole_Pad, MountingHole:MountingHole_3.2mm_M3_Pad_Via, F.Cu at (56.7, 28.1)
- added H503: MountingHole_Pad, MountingHole:MountingHole_3.2mm_M3_Pad_Via, F.Cu at (64.7, 28.1)
- added H504: MountingHole_Pad, MountingHole:MountingHole_3.2mm_M3_Pad_Via, F.Cu at (64.7, 37.3)
- added IC201: ADP2301AUJZ-R7, SnapEDA Library:SOT95P280X100-6N, F.Cu at (-26.5, -54.1)
- added IC202: ADP2301AUJZ-R7, SnapEDA Library:SOT95P280X100-6N, F.Cu at (-33.7, -49.7)
- added J201: AMASS_XT30PW-F, Connector_AMASS:AMASS_XT30PW-F_1x02_P2.50mm_Horizontal, F.Cu at (-21.9, -18.4)
- added J202: AMASS_XT30PW-M, Connector_AMASS:AMASS_XT30PW-M_1x02_P2.50mm_Horizontal, F.Cu at (-13.8, -18.4)
- added J301: SWD, Connector_PinHeader_1.27mm:PinHeader_2x05_P1.27mm_Vertical, F.Cu at (82.0, 37.6)
- added J302: USB_C_Receptacle_USB2.0, Connector_USB:USB_C_Receptacle_XKB_U262-16XN-4BVC11, F.Cu at (80.7, 24.3)
- added J401: BM04B-SURS-TFLFSN, SnapEDA Library:JST_BM04B-SURS-TF(LF)(SN), F.Cu at (-10.8, -51.8)
- added J503: TE 338069-4, SnapEDA Library:TE_338069-4, F.Cu at (10.5, -33.6)
- added JP401: SolderJumper_3_Bridged12, Jumper:SolderJumper-3_P1.3mm_Bridged12_Pad1.0x1.5mm, F.Cu at (-4.13, -52.1)
- added JP402: SolderJumper_3_Bridged12, Jumper:SolderJumper-3_P1.3mm_Bridged12_Pad1.0x1.5mm, F.Cu at (-11.9, -47.2)
- added L201: 4.7u 2.0A, SnapEDA Library:CDRH5D28RHPNP-4R7NC, F.Cu at (-18.5, -69.4)
- added L202: 15u, BluePill-Footprints:MPIT4018-150M-LF, F.Cu at (-26.3, -59.5)
- added L203: 4.7u 2.0A, SnapEDA Library:CDRH5D28RHPNP-4R7NC, F.Cu at (-40.4, -48.0)
- added Q201: AO3401A, Package_TO_SOT_SMD:SOT-23, F.Cu at (-20.1, -63.3)
- added R201: 56k, Resistor_SMD:R_0402_1005Metric, F.Cu at (-3.85, -72.3)
- added R202: 6.8k, Resistor_SMD:R_0402_1005Metric, F.Cu at (-3.85, -70.3)
- added R203: 470R, Resistor_SMD:R_0402_1005Metric, F.Cu at (-9.33, -65.3)
- added R204: 1k02, Resistor_SMD:R_0402_1005Metric, F.Cu at (-18.5, -55.6)
- added R205: 56k, Resistor_SMD:R_0402_1005Metric, F.Cu at (-21.1, -57.5)
- added R206: 10.2k, Resistor_SMD:R_0402_1005Metric, F.Cu at (-5.45, -68.3)
- added R207: 3k4, Resistor_SMD:R_0402_1005Metric, F.Cu at (-30.9, -45.9)
- added R208: 1k, Resistor_SMD:R_0402_1005Metric, F.Cu at (-23.6, -50.9)
- added R209: 1k, Resistor_SMD:R_0402_1005Metric, F.Cu at (-28.0, -45.9)
- added R210: 52.3k, Resistor_SMD:R_0402_1005Metric, F.Cu at (-18.2, -57.5)
- added R211: 10k, Resistor_SMD:R_0402_1005Metric, F.Cu at (-12.2, -63.3)
- added R212: 56k, Resistor_SMD:R_0402_1005Metric, F.Cu at (-25.7, -48.4)
- added R213: 10.2k, Resistor_SMD:R_0402_1005Metric, F.Cu at (-12.2, -65.3)
- added R301: 0R, Resistor_SMD:R_0402_1005Metric, F.Cu at (90.0, 36.9)
- added R302: 10k, Resistor_SMD:R_0402_1005Metric, F.Cu at (86.8, 42.9)
- added R303: 1k, Resistor_SMD:R_0402_1005Metric, F.Cu at (103.0, 27.0)
- added R304: 10k, Resistor_SMD:R_0402_1005Metric, F.Cu at (107.1, 22.4)
- added R305: 2k2, Resistor_SMD:R_0402_1005Metric, F.Cu at (90.0, 38.9)
- added R306: 2k2, Resistor_SMD:R_0402_1005Metric, F.Cu at (110.0, 22.4)
- added R307: 2k2, Resistor_SMD:R_0402_1005Metric, F.Cu at (92.9, 38.9)
- added R308: 2k2, Resistor_SMD:R_0402_1005Metric, F.Cu at (103.0, 29.0)
- added R309: 22R, Resistor_SMD:R_0402_1005Metric, F.Cu at (92.9, 36.9)
- added R310: 22R, Resistor_SMD:R_0402_1005Metric, F.Cu at (106.2, 25.0)
- added R311: 22R, Resistor_SMD:R_0402_1005Metric, F.Cu at (90.0, 40.9)
- added R312: 2k2, Resistor_SMD:R_0402_1005Metric, F.Cu at (73.5, 20.1)
- added R313: 2k2, Resistor_SMD:R_0402_1005Metric, F.Cu at (76.6, 18.2)
- added R401: 0R, Resistor_SMD:R_0402_1005Metric, F.Cu at (-7.60, -48.0)
- added R402: 0R, Resistor_SMD:R_0402_1005Metric, F.Cu at (-7.60, -46.0)
- added R501: 120R, Resistor_SMD:R_0402_1005Metric, F.Cu at (25.8, -36.2)
- added SW301: SW_SPDT, Button_Switch_SMD:SW_SPDT_PCM12, F.Cu at (74.9, 34.3)
- added U201: LP5907QMFX-3.3Q1, SnapEDA Library:SOT95P280X145-5N, F.Cu at (-50.2, -48.7)
- added U202: LM2842X, Package_TO_SOT_SMD:TSOT-23-6, F.Cu at (-11.9, -71.0)
- added U301: STM32F405RGT6, Package_QFP:LQFP-64_10x10mm_P0.5mm, F.Cu at (94.4, 28.7)
- added U302: USBLC6-2SC6, Package_TO_SOT_SMD:SOT-23-6, F.Cu at (72.6, 40.5)
- added U401: ICM-42670-P, SnapEDA Library:IC_ICM-42670-P, F.Cu at (53.0, 74.1)
- added U501: SN65HVD232QDRQ1, SnapEDA Library:SOIC127P599X175-8N, F.Cu at (9.64, -24.4)
- added U502: LSF0102DCUR, SnapEDA Library:SOP50P310X90-8N, F.Cu at (-42.9, -9.33)
- added Y301: 16MHz, Crystal:Crystal_SMD_3225-4Pin_3.2x2.5mm, F.Cu at (82.5, 33.6)
Routing:
- net +5V: track 24.9 -> 0.00 mm
- net VS: track 44.4 -> 26.4 mm
- net Net-(C23-Pad2): track 16.1 -> 0.00 mm, vias 2 -> 0
- net GND: track 81.9 -> 94.5 mm
- net Earth: track 12.1 -> 0.00 mm, vias 5 -> 0
- net (no net): track 0.00 -> 11.9 mm
- net Net-(C2-Pad1): track 7.56 -> 0.00 mm
- net +3V3: track 211.4 -> 217.3 mm
- net /Microcontroller/CONN_SWDIO: track 4.53 -> 0.00 mm
- net Net-(D1-Pad1): track 3.82 -> 0.00 mm
- net Net-(D1-Pad2): track 3.56 -> 0.00 mm
- net Net-(IC2-Pad4): track 2.92 -> 0.00 mm
- net Net-(R2-Pad1): track 2.84 -> 0.00 mm
- net Net-(IC2-Pad3): track 2.41 -> 0.00 mm
- net Net-(C2-Pad2): track 1.79 -> 0.00 mm
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- removed copper zone on B.Cu, net Earth

Commit message: final commit before holiday
Parts:
- removed C203: 2u2, Capacitor_SMD:C_0603_1608Metric
- removed C206, C504: 100n, Capacitor_SMD:C_0402_1005Metric
- removed C208: 10u, Capacitor_SMD:C_0603_1608Metric
- removed D201: LM5Z2V7T1G, Diode_SMD:D_SOD-523
- removed D203: B5819W, Diode_SMD:D_SOD-123
- removed D205: GREEN, LED_SMD:LED_0603_1608Metric
- removed D306: RCLAMP0521P-N, Diode_SMD:D_0402_1005Metric
- removed the D503 at (22.9, -36.2)
- removed FB201, FB501: 100R, Inductor_SMD:L_0603_1608Metric
- removed J302: USB_C_Receptacle_USB2.0, Connector_USB:USB_C_Receptacle_XKB_U262-16XN-4BVC11
- removed L202: 15u, BluePill-Footprints:MPIT4018-150M-LF
- removed Q201: AO3401A, Package_TO_SOT_SMD:SOT-23
- removed R203: 470R, Resistor_SMD:R_0402_1005Metric
- removed R204: 1k02, Resistor_SMD:R_0402_1005Metric
- removed R207: 3k4, Resistor_SMD:R_0402_1005Metric
- removed R209: 1k, Resistor_SMD:R_0402_1005Metric
- removed R312, R313: 2k2, Resistor_SMD:R_0402_1005Metric
- removed U202: LM2842X, Package_TO_SOT_SMD:TSOT-23-6
- added D307: RCLAMP0521P-N, Diode_SMD:D_0402_1005Metric, F.Cu at (33.1, 65.2)
- added D501: GREEN, LED_SMD:LED_0603_1608Metric, F.Cu at (32.8, -6.09)
- added F201: 0ZCG0050FF2C, SnapEDA Library:0ZCG0050FF2C, F.Cu at (-38.3, -41.0)
- added F202: 0ZCG0050FF2C, SnapEDA Library:0ZCG0050FF2C, F.Cu at (-28.8, -41.0)
- added J303: USB4520-03-0-A_REVA, SnapEDA Library:GCT_USB4520-03-0-A_REVA, F.Cu at (38.4, 25.6)
- added J501: Conn_01x04, SnapEDA Library:JST_B4B-XH-A(LF)(SN), F.Cu at (-7.82, -21.5)
- added J502: TE 338069-4, SnapEDA Library:TE_338069-4, F.Cu at (-14.3, -31.5)
- added J504: Conn_01x10, Connector_PinSocket_2.54mm:PinSocket_1x10_P2.54mm_Vertical, F.Cu at (-2.28, -25.1)
- added R314: 5k1, Resistor_SMD:R_0402_1005Metric, F.Cu at (36.0, 65.2)
- added R315: 5k1, Resistor_SMD:R_0402_1005Metric, F.Cu at (32.9, 67.2)
- added R501: 1k, Resistor_SMD:R_0402_1005Metric, F.Cu at (36.8, -6.17)
- J503: value TE 338069-4 -> Conn_01x10; footprint SnapEDA Library:TE_338069-4 -> Connector_PinSocket_2.54mm:PinSocket_1x10_P2.54mm_Vertical
- U502: value LSF0102DCUR -> TXS0102DCU; footprint SnapEDA Library:SOP50P310X90-8N -> Package_SO:VSSOP-8_2.3x2mm_P0.5mm
- moved C201 119.9 mm to (-4.72, 47.8)
- moved C205 117.6 mm to (-10.6, 50.1)
- moved D204 99.9 mm to (-10.3, 45.9)
- moved U201 99.4 mm to (26.4, 14.7), turned to 90 degrees
- moved R208 94.7 mm to (-10.2, 42.9)
- moved U301 77.1 mm to (17.3, 29.9)
- moved Y301 75.7 mm to (7.07, 27.3), turned to 90 degrees
- moved J503 73.7 mm to (37.7, 34.9)
- moved U401 72.4 mm to (16.9, 11.3), turned to 180 degrees
- moved locked 65.5 mm to (5.00, 55.0)
- moved U501 65.0 mm to (30.1, 37.3), turned to -90 degrees
- moved SW301 61.2 mm to (22.1, 3.40), turned to 180 degrees
- moved H501 60.9 mm to (5.00, 5.00)
- moved C503 55.2 mm to (10.6, -21.8)
- moved C302 54.8 mm to (54.0, 44.5)
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- renumbered D501 to D502, D502 to D503, R501 to R502, H503 to locked
Connections:
- net /Miscellaneous/CAN- renamed MCU_CAN2L
- C502 pad 1: /Miscellaneous/3V3_CAN -> GND
- C502 pad 2: GND -> +3V3
- D503 pad 1: /Miscellaneous/CAN+ -> MCU_CAN2H
- J503 pad 1: /Miscellaneous/3V3_CAN -> +5V
- J503 pad 2: /Miscellaneous/CAN+ -> +3V3
- J503 pad 3: GND -> MCU_CAN2H
- R401 pad 1: MCU_I2C1_SDA -> MCU_I2C2_SDA
- R402 pad 1: MCU_I2C1_SCL -> MCU_I2C2_SCL
- R502 pad 1: /Miscellaneous/CAN+ -> MCU_CAN2H
- U301 pad 14: MCU_TXD -> MCU_UART4_TX
- U301 pad 15: MCU_RXD -> MCU_UART4_RX
- U301 pad 27: IMU_INTERRUPT -> 27
- U301 pad 33: 33 -> MCU_CAN2_RX
- U301 pad 34: 34 -> MCU_CAN2_TX
- U301 pad 56: 56 -> IMU_INTERRUPT
- U401 pad 13: MCU_I2C2_SCL -> MCU_I2C1_SCL
- U401 pad 14: MCU_I2C2_SDA -> MCU_I2C1_SDA
- U501 pad 1: MCU_CAN1_TX -> MCU_CAN2_TX
- U501 pad 4: MCU_CAN1_RX -> MCU_CAN2_RX
- U501 pad 7: /Miscellaneous/CAN+ -> MCU_CAN2H
- U502 pad 1: GND -> Servo_RXD
- U502 pad 2: +3V3 -> GND
- U502 pad 3: Servo_RXD -> +3V3
- U502 pad 4: Servo_TXD -> SHIELD_UART4_RX
- U502 pad 5: MCU_TXD -> SHIELD_UART4_TX
- U502 pad 6: MCU_RXD -> +3V3
- U502 pad 8: +3V3 -> Servo_TXD
Routing:
- net +3V3: track 217.3 -> 0.00 mm, vias 7 -> 0
- net GND: track 94.5 -> 16.3 mm, vias 43 -> 13
- net /Microcontroller/MCU_BOOT0: track 28.5 -> 0.00 mm, vias 2 -> 0
- net VBUS: track 23.0 -> 0.00 mm, vias 2 -> 0
- net MCU_I2C1_SCL: track 22.5 -> 0.00 mm
- net MCU_I2C1_SDA: track 21.0 -> 0.00 mm
- net MCU_SWDIO: track 19.9 -> 0.00 mm
- net MCU_SWO: track 16.7 -> 0.00 mm
- net MCU_SWCLK: track 16.4 -> 0.00 mm
- net VS: track 26.4 -> 10.3 mm
- net IMU_INTERRUPT: track 12.2 -> 0.00 mm
- net (no net): track 11.9 -> 0.00 mm
- net MCU_CAN1_RX: track 10.6 -> 0.00 mm
- net /Microcontroller/MCU_BOOT1: track 9.37 -> 0.00 mm
- net MCU_I2C2_SDA: track 9.10 -> 0.00 mm, vias 2 -> 0
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Other:
- board size 75 x 100 mm -> 80 x 96.4 mm
- board text removed: "-"

Commit message: back from KL
Parts:
- added J505: Conn_01x10, Connector_PinSocket_2.54mm:PinSocket_1x10_P2.54mm_Vertical, F.Cu at (-37.7, -34.1)
- added J506: Conn_01x10, Connector_PinSocket_2.54mm:PinSocket_1x10_P2.54mm_Vertical, F.Cu at (2.30, 25.5)
- moved JP401 101.2 mm to (18.3, 66.1)
- moved JP402 101.2 mm to (10.6, 71.0)
- moved R401 101.2 mm to (14.9, 70.2)
- moved R402 101.2 mm to (14.9, 72.2)
- moved J401 91.8 mm to (20.2, 56.8), turned to 180 degrees
- moved C301 68.5 mm to (9.04, 17.6)
- moved R301 64.3 mm to (7.63, 21.8)
- moved R302 63.9 mm to (21.6, 8.43)
- moved C302 55.4 mm to (5.14, 18.4)
- moved C502 11.1 mm to (4.07, -10.8)
- moved C503 11.1 mm to (4.07, -12.8)
Routing:
- net GND: track 16.3 -> 19.5 mm
