File: BluePill.kicad_pcb (KiCad board)
At the start: 2 copper layers, 80 x 96.4 mm, 95 parts, among them IC201 ADP2301AUJZ-R7, IC202 ADP2301AUJZ-R7, J201 AMASS_XT30PW-F, J202 AMASS_XT30PW-M, J301 SWD, J303 USB4520-03-0-A_REVA, J401 BM04B-SURS-TFLFSN, J501 Conn_01x04, J502 TE 338069-4, J503 Conn_01x10, J504 Conn_01x10, J505 Conn_01x10, J506 Conn_01x10, SW301 SW_SPDT, U201 LP5907QMFX-3.3Q1, U301 STM32F405RGT6, U302 USBLC6-2SC6, U401 ICM-42670-P, U501 SN65HVD232QDRQ1, U502 TXS0102DCU, Y301 16MHz

Commit message: sdioghoasidgn
Parts:
- removed D307: RCLAMP0521P-N, Diode_SMD:D_0402_1005Metric
- moved U401 5.24 mm to (17.9, 16.4)
- moved C301 2.74 mm to (11.3, 19.1)
- moved R301 2.74 mm to (9.93, 23.3)
- moved C302 2.74 mm to (7.43, 19.9)
- moved L201 0.97 mm to (-46.9, -66.6)
- moved U302 0.97 mm to (28.1, 26.2)
- moved U301 0.91 mm to (17.3, 29.0)
Connections:
- J303 pad A4_B9: VBUS -> unconnected-(J303-PadA4_B9)
- J303 pad B4_A9: VBUS -> unconnected-(J303-PadB4_A9)
Routing:
- net MCU_USB_D-: track 0.00 -> 4.58 mm
- net MCU_USB_D+: track 0.00 -> 4.58 mm

Commit message: sdgihisodgn
Parts:
- added D307: RCLAMP0521P-N, Diode_SMD:D_0402_1005Metric, F.Cu at (46.4, 23.1)
- added R312: 2k2, Resistor_SMD:R_0402_1005Metric, F.Cu at (49.3, 23.1)
- added R313: 2k2, Resistor_SMD:R_0402_1005Metric, F.Cu at (46.1, 25.1)
- added R316: 2k2, Resistor_SMD:R_0402_1005Metric, F.Cu at (49.1, 25.1)
- added R317: 2k2, Resistor_SMD:R_0402_1005Metric, F.Cu at (52.2, 23.1)
Connections:
- J303 pad A4_B9: unconnected-(J303-PadA4_B9) -> VBUS
- J303 pad B4_A9: unconnected-(J303-PadB4_A9) -> VBUS
- U301 pad 40: 40 -> MCU_I2C3_SDA
- U301 pad 41: 41 -> MCU_I2C3_SCL

Commit message: sIODGNIOSGDIONSHD
Parts:
- removed D307: RCLAMP0521P-N, Diode_SMD:D_0402_1005Metric
- removed J303: USB4520-03-0-A_REVA, SnapEDA Library:GCT_USB4520-03-0-A_REVA
- removed R313: 2k2, Resistor_SMD:R_0402_1005Metric
- removed the R314 at (36.0, 65.2)
- removed the R315 at (32.9, 67.2)
- removed the R316 at (49.1, 25.1)
- added D306: RCLAMP0521P-N, Diode_SMD:D_0402_1005Metric, F.Cu at (44.5, 25.7)
- added J302: USB4085-GF-A_REVA4, SnapEDA Library:GCT_USB4085-GF-A_REVA4, F.Cu at (35.5, 26.6)
- added J507: Conn_02x05_Odd_Even, Connector_PinSocket_2.54mm:PinSocket_2x05_P2.54mm_Vertical, F.Cu at (2.38, 11.7)
- added J508: Conn_02x05_Odd_Even, Connector_PinSocket_2.54mm:PinSocket_2x05_P2.54mm_Vertical, F.Cu at (16.3, 11.8)
- added R304: 5k1, Resistor_SMD:R_0402_1005Metric, F.Cu at (47.4, 25.7)
- added R305: 5k1, Resistor_SMD:R_0402_1005Metric, F.Cu at (44.3, 27.7)
- moved U201 32.4 mm to (26.5, 47.1)
- moved U401 27.2 mm to (15.5, 43.5)
- moved C301 14.1 mm to (-2.71, 20.1)
- moved C302 14.1 mm to (-6.60, 20.9)
- moved R302 14.1 mm to (-4.11, 24.4)
- moved R307 7.28 mm to (48.9, 16.6)
- moved R301 7.28 mm to (46.0, 16.6)
- moved R402 4.53 mm to (19.2, 70.8)
- moved J401 1.22 mm to (19.0, 57.2)
- renumbered R312 to R301, R301 to R302, R302 to R303, R303 to R306, R317 to R307, R304 to R308, R305 to R309, R306 to R310, R307 to R311, R308 to R312, R309 to R314, R310 to R315, R311 to R316
Routing:
- net VBUS: track 0.00 -> 15.0 mm
- net GND: track 19.5 -> 27.1 mm
- net CONN_USB_D-: track 0.00 -> 4.04 mm
Other:
- outline, holes or cut-outs redrawn

Commit message: asdbuioasdbgaseni
Connections:
- J505 pad 1: unconnected-(J505-Pad1) -> +3V3
- J505 pad 10: unconnected-(J505-Pad10) -> GND
- J507 pad 1: unconnected-(J507-Pad1) -> +3V3
- J507 pad 2: unconnected-(J507-Pad2) -> MCU_CAN1_TX
- J507 pad 3: unconnected-(J507-Pad3) -> GND
- J507 pad 4: unconnected-(J507-Pad4) -> MCU_CAN1_RX

Commit message: sdiognsidognsdb
Parts:
- added J509: Conn_01x05, Connector_PinSocket_2.54mm:PinSocket_1x05_P2.54mm_Vertical, F.Cu at (-16.5, -2.30)
- added J510: Conn_01x05, Connector_PinSocket_2.54mm:PinSocket_1x05_P2.54mm_Vertical, F.Cu at (23.5, 57.7)
- moved R303 21.0 mm to (42.6, 9.53)
- moved H502 17.2 mm to (52.2, 4.47)
- moved R402 17.1 mm to (14.5, 54.3), turned to -90 degrees
- moved JP402 16.8 mm to (11.5, 54.2)
- moved R401 16.0 mm to (15.8, 54.3), turned to -90 degrees
- moved J501 13.2 mm to (-4.45, -34.3)
- moved JP401 11.9 mm to (18.9, 54.2)
- moved SW301 9.59 mm to (15.8, 10.6)
- moved J301 7.27 mm to (32.2, 17.1), turned to 90 degrees
- moved H501 5.88 mm to (5.00, 10.9)
- moved J507 5.23 mm to (2.33, 16.9)
- moved IC201 4.28 mm to (-12.8, -21.4)
- moved J508 4.23 mm to (17.1, 15.9)
- moved J401 3.90 mm to (15.2, 57.8)
- moved U502 3.01 mm to (-8.20, -14.0)
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Connections:
- D501 pad 2: /Miscellaneous/SHIELD_STAT_LED -> 35
- J503 pad 9: 57 -> 35
- J504 pad 9: /Miscellaneous/SHIELD_STAT_LED -> 35
- J505 pad 1: +3V3 -> +5V
- J505 pad 2: unconnected-(J505-Pad2) -> +3V3
- J506 pad 1: unconnected-(J506-Pad1) -> +5V
- J506 pad 10: unconnected-(J506-Pad10) -> GND
- J506 pad 7: unconnected-(J506-Pad7) -> SPI1_SCK
- J506 pad 8: unconnected-(J506-Pad8) -> SPI1_MISO
- J506 pad 9: unconnected-(J506-Pad9) -> SPI1_MOSI
- J507 pad 10: unconnected-(J507-Pad10) -> MCU_CAN1_RX
- J507 pad 2: MCU_CAN1_TX -> 16
- J507 pad 4: MCU_CAN1_RX -> 11
- J507 pad 5: unconnected-(J507-Pad5) -> 9
- J507 pad 6: unconnected-(J507-Pad6) -> 10
- J507 pad 7: unconnected-(J507-Pad7) -> 8
- J507 pad 8: unconnected-(J507-Pad8) -> MCU_CAN1_TX
- J507 pad 9: unconnected-(J507-Pad9) -> 4
- J508 pad 1: unconnected-(J508-Pad1) -> +3V3
- J508 pad 10: unconnected-(J508-Pad10) -> 35
- J508 pad 2: unconnected-(J508-Pad2) -> 2
- J508 pad 3: unconnected-(J508-Pad3) -> GND
- J508 pad 4: unconnected-(J508-Pad4) -> 3
- J508 pad 5: unconnected-(J508-Pad5) -> 35
- J508 pad 6: unconnected-(J508-Pad6) -> 35
- J508 pad 7: unconnected-(J508-Pad7) -> 35
- J508 pad 8: unconnected-(J508-Pad8) -> 35
- J508 pad 9: unconnected-(J508-Pad9) -> 35
- U301 pad 21: 21 -> SPI1_SCK
- U301 pad 22: 22 -> SPI1_MISO
- U301 pad 23: 23 -> SPI1_MOSI
- U301 pad 27: 27 -> IMU_INTERRUPT
- U301 pad 35: 35 -> SHIELD_STAT_LED
- U301 pad 56: IMU_INTERRUPT -> 56
Routing:
- net VBUS: track 15.0 -> 2.70 mm
- net GND: track 27.1 -> 20.5 mm

Commit message: sdgnseiogniosegn
Parts:
- moved J507 31.7 mm to (-29.3, 16.9)
- moved C202 30.5 mm to (-76.6, -46.4)
- moved C204 30.5 mm to (-74.4, -56.8)
- moved C209 30.5 mm to (-76.6, -48.6)
- moved F201 30.5 mm to (-68.8, -39.7)
- moved R206 30.5 mm to (-64.2, -63.3)
- moved F202 30.5 mm to (-59.3, -39.7)
- moved C207 30.5 mm to (-64.9, -57.1)
- moved C210 30.5 mm to (-59.6, -46.9)
- moved C211 30.5 mm to (-64.8, -44.9)
- moved D202 30.5 mm to (-63.3, -52.8)
- moved D206 30.5 mm to (-78.7, -51.9)
- moved L201 30.5 mm to (-77.4, -65.4)
- moved L203 30.5 mm to (-70.9, -46.7)
- moved R201 30.5 mm to (-62.5, -67.3)
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Connections:
- net SHIELD_I2C1_SCL renamed SHIELD_I2C2_SDA
- J503 pad 10: GND -> 35
- J503 pad 3: MCU_CAN2H -> GND
- J503 pad 4: MCU_CAN2L -> MCU_CAN2H
- J503 pad 5: MCU_UART4_TX -> MCU_CAN2L
- J503 pad 6: MCU_UART4_RX -> MCU_UART4_TX
- J503 pad 7: MCU_I2C1_SDA -> MCU_UART4_RX
- J503 pad 8: MCU_I2C1_SCL -> MCU_I2C2_SDA
- J503 pad 9: 35 -> MCU_I2C2_SCL
- J504 pad 10: GND -> 35
- J504 pad 3: SHIELD_CAN2H -> GND
- J504 pad 4: SHIELD_CAN2L -> SHIELD_CAN2H
- J504 pad 5: SHIELD_UART4_TX -> SHIELD_CAN2L
- J504 pad 6: SHIELD_UART4_RX -> SHIELD_UART4_TX
- J504 pad 7: SHIELD_I2C1_SDA -> SHIELD_UART4_RX
- J504 pad 9: 35 -> SHIELD_I2C2_SCL
- J506 pad 10: GND -> MCU_SPI1_MOSI
- J506 pad 2: unconnected-(J506-Pad2) -> +3V3
- J506 pad 3: unconnected-(J506-Pad3) -> GND
- J506 pad 4: unconnected-(J506-Pad4) -> MCU_CAN1_TX
- J506 pad 5: unconnected-(J506-Pad5) -> MCU_CAN1_RX
- J506 pad 6: unconnected-(J506-Pad6) -> MCU_I2C3_SCL
- J506 pad 7: SPI1_SCK -> MCU_I2C_SDA
- J506 pad 8: SPI1_MISO -> MCU__SPI1_SCK
- J506 pad 9: SPI1_MOSI -> MCU_SPI1_MISO
- J507 pad 10: MCU_CAN1_RX -> unconnected-(J507-Pad10)
- J507 pad 8: MCU_CAN1_TX -> unconnected-(J507-Pad8)
- U301 pad 21: SPI1_SCK -> MCU_SPI1_SCK
- U301 pad 22: SPI1_MISO -> MCU_SPI1_MISO
- U301 pad 23: SPI1_MOSI -> MCU_SPI1_MOSI
Routing:
- net VS: track 10.3 -> 18.8 mm
Other:
- board size 80 x 96.4 mm -> 80 x 105 mm

Commit message: oenbioernb
Parts:
- removed H504, locked: MountingHole_Pad, MountingHole:MountingHole_3.2mm_M3_Pad_Via
- removed J507, J508: Conn_02x05_Odd_Even, Connector_PinSocket_2.54mm:PinSocket_2x05_P2.54mm_Vertical
- IC201, IC202: footprint SnapEDA Library:SOT95P280X100-6N -> BM04B:SOT95P280X100-6N
- moved C202 91.1 mm to (13.6, -33.8)
- moved C204 91.1 mm to (15.8, -44.1)
- moved C207 91.1 mm to (25.3, -44.4)
- moved C209 91.1 mm to (13.6, -35.9)
- moved C210 91.1 mm to (30.5, -34.2)
- moved C211 91.1 mm to (25.3, -32.3)
- moved D202 91.1 mm to (26.9, -40.2)
- moved D206 91.1 mm to (11.5, -39.2)
- moved F201 91.1 mm to (21.3, -27.1)
- moved F202 91.1 mm to (30.8, -27.1)
- moved L201 91.1 mm to (12.8, -52.7)
- moved L203 91.1 mm to (19.3, -34.1)
- moved R201 91.1 mm to (27.6, -54.6)
- moved R202 91.1 mm to (27.6, -52.7)
- moved R205 91.1 mm to (26.0, -46.9)
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Connections:
- J503 pad 8: MCU_I2C2_SDA -> MCU_USART3_TX
- J503 pad 9: MCU_I2C2_SCL -> MCU_USART3_RX
- J504 pad 8: SHIELD_I2C2_SDA -> MCU_USART3_TX
- J504 pad 9: SHIELD_I2C2_SCL -> MCU_USART3_RX
- J505 pad 1: +5V -> unconnected-(J505-Pad1)
- J505 pad 10: GND -> unconnected-(J505-Pad10)
- J505 pad 2: +3V3 -> unconnected-(J505-Pad2)
- J506 pad 6: MCU_I2C3_SCL -> MCU_I2C1_SCL
- J506 pad 7: MCU_I2C_SDA -> MCU_I2C1_SDA
- J510 pad 1: unconnected-(J510-Pad1) -> 20
- J510 pad 2: unconnected-(J510-Pad2) -> 24
- J510 pad 3: unconnected-(J510-Pad3) -> 25
- J510 pad 4: unconnected-(J510-Pad4) -> 26
- J510 pad 5: unconnected-(J510-Pad5) -> 42
- U301 pad 51: 51 -> MCU_USART3_TX
- U301 pad 52: 52 -> MCU_USART3_RX
- U401 pad 13: MCU_I2C1_SCL -> MCU_I2C3_SCL
- U401 pad 14: MCU_I2C1_SDA -> MCU_I2C3_SDA
Routing:
- net MCU_USB_D-: track 4.58 -> 0.00 mm
- net MCU_USB_D+: track 4.58 -> 0.00 mm
- net VS: track 18.8 -> 16.6 mm
Other:
- board size 80 x 105 mm -> 80 x 95 mm
- board text added: "H"
- board text added: "L"
- board text removed: "+"

Commit message: sepbmwebp
Parts:
- moved J502 36.8 mm to (-28.1, -22.0)
- moved IC201 5.71 mm to (-31.4, -9.85)
- moved J301 5.00 mm to (26.9, 4.80)
- moved SW301 5.00 mm to (6.60, 3.55)
- moved H501 5.00 mm to (35.0, 5.00)
- moved H502 5.00 mm to (5.00, 40.0)
- moved J302 5.00 mm to (28.8, 40.5)
- moved J401 5.00 mm to (15.2, 42.8)
- moved J503 5.00 mm to (37.7, 19.9)
- moved J506 5.00 mm to (2.30, 10.5)
- moved JP401 5.00 mm to (18.9, 39.2)
- moved JP402 5.00 mm to (11.5, 39.2)
- moved R303 5.00 mm to (7.50, 8.42)
- moved R401 5.00 mm to (15.8, 39.3)
- moved R402 5.00 mm to (14.5, 39.3)
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Other:
- board size 80 x 95 mm -> 80 x 90 mm
