File: BluePill.kicad_pcb (KiCad board)
At the start: 2 copper layers, 80 x 90 mm, 97 parts, among them IC201 ADP2301AUJZ-R7, IC202 ADP2301AUJZ-R7, J201 AMASS_XT30PW-F, J202 AMASS_XT30PW-M, J301 SWD, J302 USB4085-GF-A_REVA4, J401 BM04B-SURS-TFLFSN, J501 Conn_01x04, J502 TE 338069-4, J503 Conn_01x10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

Commit message: sidbnb
Parts:
- removed J509, J510: Conn_01x05, Connector_PinSocket_2.54mm:PinSocket_1x05_P2.54mm_Vertical
- J505, J506: value Conn_01x10 -> Conn_01x13; footprint Connector_PinSocket_2.54mm:PinSocket_1x10_P2.54mm_Vertical -> Connector_PinSocket_2.54mm:PinSocket_1x13_P2.54mm_Vertical
- moved J506 66.6 mm to (-37.7, -42.7)
- moved J505 54.1 mm to (2.30, 2.30)
- moved SW301 3.70 mm to (10.3, 3.48)
- moved R303 3.70 mm to (11.2, 8.39)
- moved J301 1.17 mm to (26.3, 3.80)
Connections:
- J505 pad 10: unconnected-(J505-Pad10) -> MCU_SPI1_MOSI
- J505 pad 4: unconnected-(J505-Pad4) -> MCU_CAN1_TX
- J505 pad 5: unconnected-(J505-Pad5) -> MCU_CAN1_RX
- J505 pad 6: unconnected-(J505-Pad6) -> MCU_I2C1_SCL
- J505 pad 7: unconnected-(J505-Pad7) -> MCU_I2C1_SDA
- J505 pad 8: unconnected-(J505-Pad8) -> MCU__SPI1_SCK
- J505 pad 9: unconnected-(J505-Pad9) -> MCU_SPI1_MISO
- J506 pad 10: MCU_SPI1_MOSI -> unconnected-(J506-Pad10)
- J506 pad 4: MCU_CAN1_TX -> unconnected-(J506-Pad4)
- J506 pad 5: MCU_CAN1_RX -> unconnected-(J506-Pad5)
- J506 pad 6: MCU_I2C1_SCL -> unconnected-(J506-Pad6)
- J506 pad 7: MCU_I2C1_SDA -> unconnected-(J506-Pad7)
- J506 pad 8: MCU__SPI1_SCK -> unconnected-(J506-Pad8)
- J506 pad 9: MCU_SPI1_MISO -> unconnected-(J506-Pad9)

Commit message: sdighsidgh
Parts:
- IC201, IC202: footprint BM04B:SOT95P280X100-6N -> SnapEDA Library:SOT95P280X100-6N
- J302: value USB4085-GF-A_REVA4 -> USB4110-GF-A_REVB; footprint SnapEDA Library:GCT_USB4085-GF-A_REVA4 -> SnapEDA Library:GCT_USB4110-GF-A_REVB
- moved R304 16.6 mm to (36.9, 38.5)
- moved D306 13.1 mm to (37.1, 36.5)
- moved R305 9.79 mm to (40.0, 36.5)
- moved J302 2.06 mm to (28.4, 38.5)
- moved U302 0.85 mm to (28.4, 33.3)
Connections:
- R305 pad 1: GND -> Net-(J302-PadB5)
- R305 pad 2: Net-(J302-PadB5) -> GND
Routing:
- net MCU_USB_D+: track 0.00 -> 16.5 mm
- net MCU_USB_D-: track 0.00 -> 15.7 mm
- net CONN_USB_D+: track 0.00 -> 4.95 mm
- net VBUS: track 2.70 -> 0.00 mm
- net CONN_USB_D-: track 4.04 -> 5.49 mm
- net GND: track 20.5 -> 19.5 mm

Commit message: sdgnivvsdvinsv
Parts:
- J502: value TE 338069-4 -> Conn_01x02; footprint SnapEDA Library:TE_338069-4 -> SnapEDA Library:JST_B2B-XH-A(LF)(SN)
- moved R309 74.0 mm to (16.7, -2.05)
- moved R311 74.0 mm to (19.6, -2.05)
- moved C201 69.3 mm to (52.2, 8.34)
- moved C205 69.3 mm to (46.3, 10.6)
- moved R316 64.5 mm to (21.6, 8.26), turned to 90 degrees
- moved D302 63.2 mm to (29.2, -1.68)
- moved D303 60.4 mm to (22.7, 8.26), turned to -90 degrees
- moved R314 59.6 mm to (27.3, 8.36), turned to 90 degrees
- moved D304 57.6 mm to (25.0, 8.27), turned to -90 degrees
- moved R307 55.6 mm to (-3.77, 34.6)
- moved R301 53.8 mm to (-3.67, 37.4)
- moved C307 51.5 mm to (24.2, 27.9)
- moved D204 49.5 mm to (34.4, 24.6), turned to -90 degrees
- moved R208 49.2 mm to (34.5, 22.3), turned to 180 degrees
- moved C306 46.7 mm to (26.3, 16.0), turned to 90 degrees
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Connections:
- J502 pad 1: unconnected-(J502-Pad1) -> SHIELD_CAN2L
- J505 pad 8: MCU__SPI1_SCK -> MCU_SPI1_SCK
- U301 pad 17: 17 -> unconnected-(U301-Pad17)
- U301 pad 2: 2 -> unconnected-(U301-Pad2)
- U301 pad 20: 20 -> unconnected-(U301-Pad20)
- U301 pad 24: 24 -> unconnected-(U301-Pad24)
- U301 pad 25: 25 -> unconnected-(U301-Pad25)
- U301 pad 26: 26 -> unconnected-(U301-Pad26)
- U301 pad 3: 3 -> unconnected-(U301-Pad3)
- U301 pad 37: 37 -> unconnected-(U301-Pad37)
- U301 pad 38: 38 -> unconnected-(U301-Pad38)
- U301 pad 39: 39 -> unconnected-(U301-Pad39)
- U301 pad 4: 4 -> unconnected-(U301-Pad4)
- U301 pad 42: 42 -> unconnected-(U301-Pad42)
- U301 pad 43: 43 -> unconnected-(U301-Pad43)
- U301 pad 50: 50 -> unconnected-(U301-Pad50)
- U301 pad 53: 53 -> unconnected-(U301-Pad53)
- U301 pad 54: 54 -> unconnected-(U301-Pad54)
- U301 pad 56: 56 -> unconnected-(U301-Pad56)
- U301 pad 57: 57 -> unconnected-(U301-Pad57)
- U301 pad 8: 8 -> unconnected-(U301-Pad8)
- U301 pad 9: 9 -> unconnected-(U301-Pad9)
Routing:
- net +3V3: track 0.00 -> 32.4 mm
- net GND: track 19.5 -> 41.7 mm, vias 13 -> 22
- net MCU_CAN2L: track 0.00 -> 17.0 mm
- net MCU_CAN2H: track 0.00 -> 15.8 mm
- net MCU_CAN2_TX: track 0.00 -> 15.1 mm, vias 0 -> 2
- net MCU_CAN2_RX: track 0.00 -> 14.5 mm, vias 0 -> 2
- net MCU_SWDIO: track 0.00 -> 12.4 mm
- net /Microcontroller/MCU_BOOT0: track 0.00 -> 11.8 mm
- net MCU_I2C2_SDA: track 0.00 -> 9.93 mm
- net +5V: track 0.00 -> 9.85 mm
- net MCU_I2C2_SCL: track 0.00 -> 9.60 mm
- net MCU_SWO: track 0.00 -> 8.16 mm
- net MCU_SWCLK: track 0.00 -> 7.85 mm
- net /Microcontroller/MCU_BOOT1: track 0.00 -> 7.27 mm, vias 0 -> 2
- net /Microcontroller/MCU_HSE_IN: track 0.00 -> 7.13 mm
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
Commit message: ormbroermbo
Parts:
- moved C311 1.68 mm to (56.5, 31.1)
- moved C312 0.96 mm to (31.3, 35.9), turned to 180 degrees
- moved C303 0.54 mm to (49.4, 33.5)
Changed lines of the file:
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@@
   )
   (footprint "Capacitor_SMD:C_0402_1005Metric" (layer "F.Cu")
-    (at 32.045 35.24)
+    (at 31.3 35.85 180)
     (descr "Capacitor SMD 0402 (1005 Metric), square (rectangular) end terminal, IPC_7351 nominal, (Body size source: IPC-SM-782 page 76, https://www.pcb-3d.com/wordpress/wp-content/uploads/ipc-sm-782a_amendment_1_and_2.pdf), generated with kicad-footprint-generator")
     (tags "capacitor")
@@
     (property "Sheetname" "Microcontroller")
     (attr smd)
-    (fp_text reference "C312" (at 0 -1.16) (layer "F.SilkS")
+    (fp_text reference "C312" (at -1.3 1.3) (layer "F.SilkS") hide
       (effects (font (size 1 1) (thickness 0.15)))
     )
@@
     (fp_line (start 0.5 0.25) (end -0.5 0.25) (layer "F.Fab") (width 0.1))
     (fp_line (start 0.5 -0.25) (end 0.5 0.25) (layer "F.Fab") (width 0.1))
-    (pad "1" smd roundrect (at -0.48 0) (size 0.56 0.62) (layers "F.Cu" "F.Paste" "F.Mask") (roundrect_rratio 0.25)
+    (pad "1" smd roundrect (at -0.48 0 180) (size 0.56 0.62) (layers "F.Cu" "F.Paste" "F.Mask") (roundrect_rratio 0.25)
       (net 1 "GND") (pintype "passive"))
-    (pad "2" smd roundrect (at 0.48 0) (size 0.56 0.62) (layers "F.Cu" "F.Paste" "F.Mask") (roundrect_rratio 0.25)
+    (pad "2" smd roundrect (at 0.48 0 180) (size 0.56 0.62) (layers "F.Cu" "F.Paste" "F.Mask") (roundrect_rratio 0.25)
       (net 8 "VBUS") (pintype "passive"))
     (model "${KICAD6_3DMODEL_DIR}/Capacitor_SMD.3dshapes/C_0402_1005Metric.wrl"
@@
   )
   (footprint "Capacitor_SMD:C_0402_1005Metric" (layer "F.Cu")
-    (at 58.015 31.815)
+    (at 56.5 31.1)
     (descr "Capacitor SMD 0402 (1005 Metric), square (rectangular) end terminal, IPC_7351 nominal, (Body size source: IPC-SM-782 page 76, https://www.pcb-3d.com/wordpress/wp-content/uploads/ipc-sm-782a_amendment_1_and_2.pdf), generated with kicad-footprint-generator")
     (tags "capacitor")
@@
   )
   (footprint "Capacitor_SMD:C_0603_1608Metric" (layer "F.Cu")
-    (at 49.83 33.745)
+    (at 49.375 33.45)
     (descr "Capacitor SMD 0603 (1608 Metric), square (rectangular) end terminal, IPC_7351 nominal, (Body size source: IPC-SM-782 page 76, https://www.pcb-3d.com/wordpress/wp-content/uploads/ipc-sm-782a_amendment_1_and_2.pdf), generated with kicad-footprint-generator")
     (tags "capacitor")

Commit message: sdojbmosbm
Parts:
- moved R305 14.2 mm to (31.9, 33.8), turned to 90 degrees
- moved D306 13.2 mm to (32.2, 35.3)
- moved R304 12.7 mm to (25.4, 35.2)
- moved C312 3.04 mm to (30.8, 32.9), turned to 90 degrees
Routing:
- net GND: track 41.7 -> 67.2 mm, vias 22 -> 26
- net VBUS: track 0.00 -> 19.8 mm, vias 0 -> 3
- net Net-(J302-PadB5): track 0.00 -> 3.94 mm
- net Net-(J302-PadA5): track 0.00 -> 2.75 mm

Commit message: dinbdiofbn
Parts:
- moved C402 66.6 mm to (-2.13, 36.0)
- moved C403 66.6 mm to (-2.13, 38.0)
- moved C401 53.3 mm to (8.87, 34.2)
- moved C309 49.0 mm to (12.9, 16.3), turned to 90 degrees
- moved C311 46.4 mm to (10.6, 23.8), turned to 90 degrees
- moved C310 44.0 mm to (14.8, 14.3)
- moved C303 41.3 mm to (11.4, 17.2), turned to 90 degrees
- moved D503 23.8 mm to (44.6, 13.8)
- moved R502 23.8 mm to (46.1, 16.9)
- moved D502 23.8 mm to (42.0, 17.0)
- moved C205 21.6 mm to (31.7, 26.5)
- moved C501 21.3 mm to (30.9, 12.0), turned to 180 degrees
- moved C201 21.0 mm to (34.7, 19.9), turned to -90 degrees
- moved R301 18.0 mm to (14.1, 34.3), turned to -90 degrees
- moved R307 17.9 mm to (14.1, 36.3), turned to 90 degrees
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Connections:
- J505 pad 2: unconnected-(J505-Pad2) -> +3V3
- J505 pad 4: MCU_CAN1_TX -> MCU_CAN1_RX
- J505 pad 5: MCU_CAN1_RX -> MCU_CAN1_TX
- J506 pad 2: +3V3 -> unconnected-(J506-Pad2)
Routing:
- net +3V3: track 32.4 -> 266.8 mm, vias 0 -> 4
- net MCU_UART4_TX: track 0.00 -> 35.6 mm, vias 0 -> 2
- net MCU_UART4_RX: track 0.00 -> 35.2 mm, vias 0 -> 2
- net MCU_I2C1_SCL: track 0.00 -> 25.0 mm
- net GND: track 67.2 -> 91.9 mm, vias 26 -> 35
- net MCU_I2C1_SDA: track 0.00 -> 23.1 mm
- net MCU_SPI1_SCK: track 0.00 -> 22.0 mm
- net MCU_SPI1_MISO: track 0.00 -> 21.8 mm
- net MCU_SPI1_MOSI: track 0.00 -> 21.7 mm
- net MCU_CAN1_RX: track 0.00 -> 20.0 mm, vias 0 -> 2
- net MCU_CAN1_TX: track 0.00 -> 18.0 mm, vias 0 -> 2
- net 11: track 0.00 -> 17.3 mm, vias 0 -> 2
- net 16: track 0.00 -> 15.1 mm, vias 0 -> 2
- net 10: track 0.00 -> 14.1 mm, vias 0 -> 2
- net IMU_INTERRUPT: track 0.00 -> 12.9 mm
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
Commit message: digndfign
Parts:
- moved C202 79.9 mm to (-64.0, -14.7)
- moved C204 79.9 mm to (-61.8, -25.1)
- moved C207 79.9 mm to (-52.3, -25.3)
- moved C209 79.9 mm to (-64.0, -16.9)
- moved C210 79.9 mm to (-47.0, -15.2)
- moved C211 79.9 mm to (-52.2, -13.2)
- moved D202 79.9 mm to (-50.7, -21.1)
- moved D206 79.9 mm to (-66.1, -20.2)
- moved F201 79.9 mm to (-56.2, -8.00)
- moved F202 79.9 mm to (-46.7, -8.00)
- moved L201 79.9 mm to (-64.8, -33.6)
- moved L203 79.9 mm to (-58.3, -15.0)
- moved R201 79.9 mm to (-50.0, -35.6)
- moved R202 79.9 mm to (-50.0, -33.6)
- moved R205 79.9 mm to (-51.6, -27.8)
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Connections:
- D501 pad 2: 35 -> Net-(D501-Pad2)
- J503 pad 10: 35 -> SHIELD_STAT_LED
- J504 pad 10: 35 -> Net-(D501-Pad2)
- J504 pad 8: MCU_USART3_TX -> unconnected-(J504-Pad8)
- J504 pad 9: MCU_USART3_RX -> unconnected-(J504-Pad9)
Routing:
- net +5V: track 9.85 -> 81.8 mm, vias 0 -> 2
- net MCU_USART3_RX: track 0.00 -> 31.4 mm, vias 0 -> 2
- net MCU_USART3_TX: track 0.00 -> 31.1 mm, vias 0 -> 2
- net MCU_I2C3_SCL: track 0.00 -> 27.8 mm, vias 0 -> 2
- net SHIELD_CAN2L: track 0.00 -> 26.8 mm
- net SHIELD_CAN2H: track 0.00 -> 26.1 mm
- net SHIELD_STAT_LED: track 0.00 -> 25.8 mm, vias 0 -> 2
- net MCU_I2C3_SDA: track 0.00 -> 25.5 mm, vias 0 -> 2
- net +3V3: track 266.8 -> 284.1 mm, vias 4 -> 8
- net /Microcontroller/MCU_LED_A: track 0.00 -> 15.2 mm, vias 0 -> 2
- net Servo_RXD: track 0.00 -> 14.2 mm
- net Servo_TXD: track 0.00 -> 12.0 mm
- net GND: track 91.9 -> 103.9 mm, vias 35 -> 40
- net SHIELD_UART4_RX: track 0.00 -> 8.33 mm
- net MCU_CAN2L: track 18.0 -> 25.2 mm
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Other:
- board text added: "RX"
- board text added: "TX"
- board text added: "USART"

Commit message: irdshboidrehonb
Parts:
- IC201, IC202: footprint SnapEDA Library:SOT95P280X100-6N -> BM04B:SOT95P280X100-6N
- moved F202 53.7 mm to (-30.1, -59.1)
- moved C209 52.2 mm to (-35.5, -60.5)
- moved L203 42.9 mm to (-35.2, -51.1)
- moved R212 40.9 mm to (-58.7, -53.5)
- moved D206 39.9 mm to (-44.6, -53.8)
- moved L201 37.9 mm to (-32.4, -14.0), turned to 90 degrees
- moved C211 36.9 mm to (-56.9, -49.8)
- moved C210 35.2 mm to (-50.8, -50.2)
- moved F201 33.4 mm to (-24.4, -18.2)
- moved R206 31.4 mm to (-35.5, -4.65), turned to 180 degrees
- moved R202 31.2 mm to (-37.2, -5.10), turned to -90 degrees
- moved C202 31.0 mm to (-33.5, -9.60)
- moved C204 30.9 mm to (-31.6, -18.7), turned to 180 degrees
- moved R201 30.7 mm to (-37.9, -7.30), turned to -90 degrees
- moved R210 30.4 mm to (-56.9, -57.0)
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Routing:
- net VS: track 16.6 -> 20.9 mm
