File: Misc.kicad_sch (KiCad schematic)
At the start: 18 parts, among them J3 Conn_02x08_Odd_Even, J4 BM04B-SURS-TFLFSN, J5 Conn_02x04_Odd_Even, J6 Conn_02x04_Odd_Even, J7 Conn_01x05, J8 Conn_01x04, U5 SN65HVD232QDRQ1

Commit message: sdignionsrg
Parts:
- added JP1, JP2: SolderJumper_3_Bridged12, Jumper:SolderJumper-3_P1.3mm_Bridged12_Pad1.0x1.5mm, symbol Jumper:SolderJumper_3_Bridged12
- added R17, R18: 0R, Resistor_SMD:R_0402_1005Metric, symbol Device:R_Small
Connections:
- net +3V3: now also JP1.1 (A), JP2.3 (B); no longer J4.1
- net GND: now also JP1.3 (B), JP2.1 (A); no longer J4.4
- net MCU_I2C1_SCL: now also R18.1; no longer J4.3
- net MCU_I2C1_SDA: now also R17.1; no longer J4.2
- new net: J4.1, JP1.2 (C)
- new net: J4.4, JP2.2 (C)
- new net: J4.2, R17.2
- new net: J4.3, R18.2
Other:
- moved on the sheet: J3, J5, J6, J7

Commit message: siobgg:
Parts:
- removed J8: Conn_01x04, Connector_PinHeader_2.54mm:PinHeader_1x04_P2.54mm_Vertical, symbol Connector_Generic:Conn_01x04
- added J2: TE 338069-4, SnapEDA Library:TE_338069-4, symbol 338069-4:338069-4
Connections:
- net 3V3_CAN: now also J2.1
- net CAN+: now also J2.2
- net CAN-: now also J2.4
- net GND: now also J2.3
Changed lines of the file:
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@@
   (junction (at 187.96 49.53) (diameter 0) (color 0 0 0 0)
   )
+  (junction (at 229.87 44.45) (diameter 0) (color 0 0 0 0)
+  )
   (junction (at 229.87 38.1) (diameter 0) (color 0 0 0 0)
-  )
-  (junction (at 229.87 41.91) (diameter 0) (color 0 0 0 0)
   )
   (junction (at 187.96 41.91) (diameter 0) (color 0 0 0 0)
@@
     (stroke (width 0) (type default) (color 0 0 0 0))
   )
-  (wire (pts (xy 224.79 44.45) (xy 224.79 41.91))
-    (stroke (width 0) (type default) (color 0 0 0 0))
-  )
-  (wire (pts (xy 224.79 41.91) (xy 220.98 41.91))
+  (wire (pts (xy 226.06 41.91) (xy 220.98 41.91))
     (stroke (width 0) (type default) (color 0 0 0 0))
   )
@@
     (stroke (width 0) (type default) (color 0 0 0 0))
   )
-  (wire (pts (xy 229.87 38.1) (xy 229.87 41.91))
-    (stroke (width 0) (type default) (color 0 0 0 0))
-  )
   (wire (pts (xy 54.61 40.64) (xy 57.15 40.64))
     (stroke (width 0) (type default) (color 0 0 0 0))
@@
     (stroke (width 0) (type default) (color 0 0 0 0))
   )
-  (wire (pts (xy 201.93 46.99) (xy 201.93 49.53))
-    (stroke (width 0) (type default) (color 0 0 0 0))
-  )
   (wire (pts (xy 200.66 102.87) (xy 199.39 102.87))
     (stroke (width 0) (type default) (color 0 0 0 0))
   )
+  (wire (pts (xy 229.87 44.45) (xy 229.87 50.8))
+    (stroke (width 0) (type default) (color 0 0 0 0))
+  )
+  (wire (pts (xy 226.06 41.91) (xy 226.06 46.99))
+    (stroke (width 0) (type default) (color 0 0 0 0))
+  )
   (wire (pts (xy 73.66 130.81) (xy 82.55 130.81))
     (stroke (width 0) (type default) (color 0 0 0 0))
   )
-  (wire (pts (xy 224.79 44.45) (xy 245.11 44.45))
-    (stroke (width 0) (type default) (color 0 0 0 0))
-  )
-  (wire (pts (xy 201.93 49.53) (xy 199.39 49.53))
+  (wire (pts (xy 199.39 49.53) (xy 233.68 49.53))
     (stroke (width 0) (type default) (color 0 0 0 0))
   )
@@
     (stroke (width 0) (type default) (color 0 0 0 0))
   )
+  (wire (pts (xy 242.57 44.45) (xy 242.57 58.42))
+    (stroke (width 0) (type default) (color 0 0 0 0))
+  )
   (polyline (pts (xy 124.46 93.98) (xy 27.94 93.98))
     (stroke (width 0) (type default) (color 0 0 0 0))
@@
     (stroke (width 0) (type default) (color 0 0 0 0))
   )
-  (wire (pts (xy 229.87 41.91) (xy 245.11 41.91))
-    (stroke (width 0) (type default) (color 0 0 0 0))
-  )
   (wire (pts (xy 199.39 104.14) (xy 199.39 102.87))
     (stroke (width 0) (type default) (color 0 0 0 0))
@@
     (stroke (width 0) (type default) (color 0 0 0 0))
   )
+  (wire (pts (xy 245.11 44.45) (xy 242.57 44.45))
+    (stroke (width 0) (type default) (color 0 0 0 0))
+  )
+  (wire (pts (xy 233.68 41.91) (xy 245.11 41.91))
+    (stroke (width 0) (type default) (color 0 0 0 0))
+  )
   (polyline (pts (xy 265.43 24.13) (xy 130.81 24.13))
     (stroke (width 0) (type default) (color 0 0 0 0))
@@
     (stroke (width 0) (type default) (color 0 0 0 0))
   )
+  (wire (pts (xy 226.06 46.99) (xy 245.11 46.99))
+    (stroke (width 0) (type default) (color 0 0 0 0))
+  )
   (polyline (pts (xy 27.94 146.05) (xy 124.46 146.05))
     (stroke (width 0) (type default) (color 0 0 0 0))
@@
     (stroke (width 0) (type default) (color 0 0 0 0))
   )
-  (wire (pts (xy 201.93 46.99) (xy 245.11 46.99))
-    (stroke (width 0) (type default) (color 0 0 0 0))
-  )
   (wire (pts (xy 199.39 96.52) (xy 200.66 96.52))
     (stroke (width 0) (type default) (color 0 0 0 0))
@@
     (stroke (width 0) (type default) (color 0 0 0 0))
   )
+  (wire (pts (xy 229.87 44.45) (xy 237.49 44.45))
+    (stroke (width 0) (type default) (color 0 0 0 0))
+  )
   (wire (pts (xy 95.25 130.81) (xy 104.14 130.81))
     (stroke (width 0) (type default) (color 0 0 0 0))
@@
     (stroke (width 0) (type default) (color 0 0 0 0))
   )
-  (wire (pts (xy 229.87 50.8) (xy 229.87 41.91))
+  (wire (pts (xy 229.87 38.1) (xy 229.87 44.45))
+    (stroke (width 0) (type default) (color 0 0 0 0))
+  )
+  (wire (pts (xy 233.68 49.53) (xy 233.68 41.91))
+    (stroke (width 0) (type default) (color 0 0 0 0))
+  )
+  (wire (pts (xy 237.49 44.45) (xy 237.49 49.53))
     (stroke (width 0) (type default) (color 0 0 0 0))
   )
@@
   (wire (pts (xy 46.99 38.1) (xy 49.53 38.1))
     (stroke (width 0) (type default) (color 0 0 0 0))
+  )
+  (wire (pts (xy 237.49 49.53) (xy 245.11 49.53))
+    (stroke (width 0) (type default) (color 0 0 0 0))
+  )
+  (label "CAN-" (at 238.76 41.91 0)
+    (effects (font (size 0.4064 0.4064)) (justify left bottom))
   )
   (label "NOTE: REVERSED CONNECTIONS DUE TO CABLE (see encoder board)"
@@
     (effects (font (size 1.27 1.27) (thickness 0.254) bold) (justify left bottom))
   )
+  (label "CAN+" (at 238.76 46.99 0)
+    (effects (font (size 0.4064 0.4064)) (justify left bottom))
+  )
   (label "CAN+" (at 182.88 41.91 0)
     (effects (font (size 0.4064 0.4064)) (justify left bottom))
@@
     (effects (font (size 0.4064 0.4064)) (justify left bottom))
   )
-  (label "3V3_CAN" (at 232.41 41.91 0)
+  (label "3V3_CAN" (at 238.76 49.53 0)
     (effects (font (size 0.4064 0.4064)) (justify left bottom))
   )
@@
     (pin "1")
   )
-  (symbol (lib_id "Connector_Generic:Conn_01x04") (at 250.19 44.45 0) (unit 1)
-    (in_bom yes) (on_board yes)
-    (property "Reference" "J8" (id 0) (at 252.222 44.6532 0)
-      (effects (font (size 1.27 1.27)) (justify left))
-    )
-    (property "Value" "Conn_01x04" (id 1) (at 252.222 46.9646 0)
-      (effects (font (size 1.27 1.27)) (justify left))
-    )
-    (property "Footprint" "Connector_PinHeader_2.54mm:PinHeader_1x04_P2.54mm_Vertical" (id 2) (at 250.19 44.45 0)
-      (effects (font (size 1.27 1.27)) hide)
-    )
-    (property "Datasheet" "~" (id 3) (at 250.19 44.45 0)
-      (effects (font (size 1.27 1.27)) hide)
-    )
-    (pin "1")
-    (pin "2")
-    (pin "3")
-    (pin "4")
-  )
   (symbol (lib_id "Device:D_TVS") (at 229.87 54.61 270) (unit 1)
     (in_bom yes) (on_board yes)
@@
     (pin "1")
   )
-  (symbol (lib_id "power:GND") (at 245.11 49.53 0) (unit 1)
-    (in_bom yes) (on_board yes)
-    (property "Reference" "#PWR061" (id 0) (at 245.11 55.88 0)
-      (effects (font (size 1.27 1.27)) hide)
-    )
-    (property "Value" "GND" (id 1) (at 245.11 53.34 0)
-      (effects (font (size 1.27 1.27)) hide)
-    )
-    (property "Footprint" "" (id 2) (at 245.11 49.53 0)
-      (effects (font (size 1.27 1.27)) hide)
-    )
-    (property "Datasheet" "" (id 3) (at 245.11 49.53 0)
-      (effects (font (size 1.27 1.27)) hide)
-    )
-    (pin "1")
-  )
   (symbol (lib_id "BluePhil-rescue:Ferrite_Bead_Small-Device") (at 226.06 38.1 270) (unit 1)
     (in_bom yes) (on_board yes)
@@
     (pin "2")
     (pin "3")
+  )
+  (symbol (lib_id "power:GND") (at 242.57 58.42 0) (unit 1)
+    (in_bom yes) (on_board yes)
+    (property "Reference" "#PWR0110" (id 0) (at 242.57 64.77 0)
+      (effects (font (size 1.27 1.27)) hide)
+    )
+    (property "Value" "GND" (id 1) (at 242.57 62.23 0)
+      (effects (font (size 1.27 1.27)) hide)
+    )
+    (property "Footprint" "" (id 2) (at 242.57 58.42 0)
+      (effects (font (size 1.27 1.27)) hide)
+    )
+    (property "Datasheet" "" (id 3) (at 242.57 58.42 0)
+      (effects (font (size 1.27 1.27)) hide)
+    )
+    (pin "1")
   )
   (symbol (lib_id "power:GND") (at 60.96 109.22 0) (unit 1)
@@
     (pin "8")
   )
+  (symbol (lib_id "338069-4:338069-4") (at 252.73 44.45 180) (unit 1)
+    (in_bom yes) (on_board yes)
+    (property "Reference" "J2" (id 0) (at 250.19 34.29 0)
+      (effects (font (size 1.27 1.27)) (justify right))
+    )
+    (property "Value" "TE 338069-4" (id 1) (at 250.19 36.83 0)
+      (effects (font (size 1.27 1.27)) (justify right))
+    )
+    (property "Footprint" "SnapEDA Library:TE_338069-4" (id 2) (at 252.73 44.45 0)
+      (effects (font (size 1.27 1.27)) (justify left bottom) hide)
+    )
+    (property "Datasheet" "" (id 3) (at 252.73 44.45 0)
+      (effects (font (size 1.27 1.27)) (justify left bottom) hide)
+    )
+    (property "STANDARD" "Manufacturer Recommendation" (id 4) (at 252.73 44.45 0)
+      (effects (font (size 1.27 1.27)) (justify left bottom) hide)
+    )
+    (property "MANUFACTURER" "TE Connectivity AMP Connectors" (id 5) (at 252.73 44.45 0)
+      (effects (font (size 1.27 1.27)) (justify left bottom) hide)
+    )
+    (property "SERIES" "Micro-MaTch" (id 6) (at 252.73 44.45 0)
+      (effects (font (size 1.27 1.27)) (justify left bottom) hide)
+    )
+    (property "POSITIONS" "14" (id 7) (at 252.73 44.45 0)
+      (effects (font (size 1.27 1.27)) (justify left bottom) hide)
+    )
+    (property "PITCH" "2.54mm" (id 8) (at 252.73 44.45 0)
+      (effects (font (size 1.27 1.27)) (justify left bottom) hide)
+    )
+    (property "VOLTAGE" "100VDC" (id 9) (at 252.73 44.45 0)
+      (effects (font (size 1.27 1.27)) (justify left bottom) hide)
+    )
+    (property "PARTREV" "H4" (id 10) (at 252.73 44.45 0)
+      (effects (font (size 1.27 1.27)) (justify left bottom) hide)
+    )
+    (pin "1")
+    (pin "2")
+    (pin "3")
+    (pin "4")
+  )
   (symbol (lib_id "Connector_Generic:Conn_01x05") (at 113.03 111.76 0) (unit 1)

Commit message: adsigjningh
Parts:
- added U8: LSF0102DCUR, SnapEDA Library:SOP50P310X90-8N, symbol LSF0102DCUR:LSF0102DCUR
- J4: footprint BM04B:BM04B-SURS-TFLFSN -> SnapEDA Library:JST_BM04B-SURS-TF(LF)(SN)
Other:
- moved on the sheet: H1, H2, H3, H4, J3, J5, J6, J7

Commit message: skgnigniogni
Parts:
- removed J4: BM04B-SURS-TFLFSN, SnapEDA Library:JST_BM04B-SURS-TF(LF)(SN), symbol BM04B:BM04B-SURS-TFLFSN
- removed JP1, JP2: SolderJumper_3_Bridged12, Jumper:SolderJumper-3_P1.3mm_Bridged12_Pad1.0x1.5mm, symbol Jumper:SolderJumper_3_Bridged12
- removed R17, R18: 0R, Resistor_SMD:R_0402_1005Metric, symbol Device:R_Small
- added J10: Conn_01x04, symbol Connector_Generic:Conn_01x04
Connections:
- net +3V3: now also U8.7 (VREF_B)
- net +5V: now also U8.2 (VREF_A)
- net GND: now also U8.1 (GND)
- net Servo_RXD: now reaches U8.3 (A1)
- net Servo_RXD: now also J10.1 (Pin_1)
- net Servo_TXD: now reaches U8.4 (A2)
- net Servo_TXD: now also J10.2 (Pin_2)
- net MCU_TXD: now reaches U8.5 (B2)
- net MCU_RXD: now reaches U8.6 (B1)
- new net Servo_GND: J10.4 (Pin_4)
- new net Servo_VDD: J10.3 (Pin_3)
Other:
- note added: "Terminating Resistor"
- moved on the sheet: J3, J5, J6, J7, R16

Commit message: sdgionbidnb
Connections:
- net +3V3: now also U8.2 (VREF_A); no longer U8.7 (VREF_B)
- net +5V: now also U8.7 (VREF_B); no longer U8.2 (VREF_A)
Changed lines of the file:
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@@
     (stroke (width 0) (type default) (color 0 0 0 0))
   )
-  (wire (pts (xy 185.42 99.06) (xy 198.12 99.06))
+  (wire (pts (xy 186.69 99.06) (xy 198.12 99.06))
     (stroke (width 0) (type default) (color 0 0 0 0))
   )
@@
     (pin "4")
   )
-  (symbol (lib_id "power:+5V") (at 185.42 99.06 0) (unit 1)
-    (in_bom yes) (on_board yes)
-    (property "Reference" "#PWR065" (id 0) (at 185.42 102.87 0)
-      (effects (font (size 1.27 1.27)) hide)
-    )
-    (property "Value" "+5V" (id 1) (at 185.42 95.25 0))
-    (property "Footprint" "" (id 2) (at 185.42 99.06 0)
-      (effects (font (size 1.27 1.27)) hide)
-    )
-    (property "Datasheet" "" (id 3) (at 185.42 99.06 0)
-      (effects (font (size 1.27 1.27)) hide)
-    )
-    (pin "1")
-  )
   (symbol (lib_id "Connector_Generic:Conn_01x05") (at 113.03 106.68 0) (unit 1)
     (in_bom yes) (on_board yes)
@@
     (pin "4")
     (pin "5")
+  )
+  (symbol (lib_id "BluePhil-rescue:+3.3V-power") (at 186.69 99.06 0) (unit 1)
+    (in_bom yes) (on_board yes)
+    (property "Reference" "#PWR065" (id 0) (at 186.69 102.87 0)
+      (effects (font (size 1.27 1.27)) hide)
+    )
+    (property "Value" "+3.3V" (id 1) (at 186.69 95.25 0))
+    (property "Footprint" "" (id 2) (at 186.69 99.06 0)
+      (effects (font (size 1.27 1.27)) hide)
+    )
+    (property "Datasheet" "" (id 3) (at 186.69 99.06 0)
+      (effects (font (size 1.27 1.27)) hide)
+    )
+    (pin "1")
   )
   (symbol (lib_id "power:+5V") (at 33.02 104.14 0) (unit 1)
@@
     (pin "1")
   )
+  (symbol (lib_id "power:+5V") (at 179.07 99.06 0) (unit 1)
+    (in_bom yes) (on_board yes)
+    (property "Reference" "#PWR064" (id 0) (at 179.07 102.87 0)
+      (effects (font (size 1.27 1.27)) hide)
+    )
+    (property "Value" "+5V" (id 1) (at 179.07 95.25 0))
+    (property "Footprint" "" (id 2) (at 179.07 99.06 0)
+      (effects (font (size 1.27 1.27)) hide)
+    )
+    (property "Datasheet" "" (id 3) (at 179.07 99.06 0)
+      (effects (font (size 1.27 1.27)) hide)
+    )
+    (pin "1")
+  )
   (symbol (lib_id "power:GND") (at 95.25 102.87 0) (unit 1)
     (in_bom yes) (on_board yes)
@@
       (effects (font (size 1.27 1.27)) hide)
     )
-    (pin "1")
-  )
-  (symbol (lib_id "BluePhil-rescue:+3.3V-power") (at 179.07 99.06 0) (unit 1)
-    (in_bom yes) (on_board yes)
-    (property "Reference" "#PWR064" (id 0) (at 179.07 102.87 0)
-      (effects (font (size 1.27 1.27)) hide)
-    )
-    (property "Value" "+3.3V" (id 1) (at 179.07 95.25 0))
-    (property "Footprint" "" (id 2) (at 179.07 99.06 0)
-      (effects (font (size 1.27 1.27)) hide)
-    )
-    (property "Datasheet" "" (id 3) (at 179.07 99.06 0)
-      (effects (font (size 1.27 1.27)) hide)
-    )

Commit message: WEBGIOWEBGIOBWEG
Parts:
- removed J10: Conn_01x04, symbol Connector_Generic:Conn_01x04
- removed J3: Conn_02x08_Odd_Even, Connector_PinHeader_2.54mm:PinHeader_2x08_P2.54mm_Vertical, symbol Connector_Generic:Conn_02x08_Odd_Even
- removed J5, J6: Conn_02x04_Odd_Even, Connector_PinHeader_2.54mm:PinHeader_2x04_P2.54mm_Vertical, symbol Connector_Generic:Conn_02x04_Odd_Even
- removed J7: Conn_01x05, Connector_PinSocket_2.54mm:PinSocket_1x05_P2.54mm_Vertical, symbol Connector_Generic:Conn_01x05
- added C503, C504: 100n, Capacitor_SMD:C_0402_1005Metric, symbol Device:C_Small
- added D?: GREEN, LED_SMD:LED_0603_1608Metric, symbol Device:LED_Small
- added J501: Servo power, symbol Connector_Generic:Conn_01x02
- added J502: Servo serial, symbol Connector_Generic:Conn_01x02
- added J? (x2): Conn_01x10, symbol Connector_Generic:Conn_01x10
- added R?: 1k, Resistor_SMD:R_0402_1005Metric, symbol Device:R_Small
- renumbered C19 to C501, C20 to C502, D10 to D501, D11 to D502, D12 to D503, FB2 to FB501, H1 to H501, H2 to H502, H3 to H503, H4 to H504, J2 to J503, R16 to R501, U5 to U501, U8 to U502
Connections:
- net +3V3: now also U502.8 (EN), C504.2
- net +5V: now also C503.2, J?.1 (Pin_1), J?.1 (Pin_1)
- net GND: now also C503.1, C504.1, J501.2 (Pin_2), J?.10 (Pin_10), J?.10 (Pin_10), R?.2
- net Servo_RXD: now also J502.1 (Pin_1)
- net Servo_TXD: now also J502.2 (Pin_2)
- new net: D?.2 (A), J?.9 (Pin_9)
- new net: D?.1 (K), R?.1
- new net Vdrive: J501.1 (Pin_1)
Other:
- note added: "CAN Transceiver"
- note added: "Inter-board: Main"
- note added: "Inter-board: Shield"
- note added: "Servo Connectors"
- note added: "UART Level Shifter"
- moved on the sheet: C501, C502, D501, D502, D503, FB501, H501, H502, H503, H504, J503, R501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

Commit message: final commit before holiday
Parts:
- removed C504: 100n, Capacitor_SMD:C_0402_1005Metric, symbol Device:C_Small
- removed D503: RCLAMP0521P-N, Diode_SMD:D_0402_1005Metric, symbol Device:D_TVS
- removed FB501: 100R, Inductor_SMD:L_0603_1608Metric, symbol BluePhil-rescue:Ferrite_Bead_Small-Device
- removed J501: Servo power, symbol Connector_Generic:Conn_01x02
- removed J502: Servo serial, symbol Connector_Generic:Conn_01x02
- removed J503: TE 338069-4, SnapEDA Library:TE_338069-4, symbol 338069-4:338069-4
- removed U502: LSF0102DCUR, SnapEDA Library:SOP50P310X90-8N, symbol LSF0102DCUR:LSF0102DCUR
- added J501: Conn_01x04, SnapEDA Library:JST_B4B-XH-A(LF)(SN), symbol Connector_Generic:Conn_01x04
- added J502: TE 338069-4, SnapEDA Library:TE_338069-4, symbol 338069-4:338069-4
- added U502: TXS0102DCU, Package_SO:VSSOP-8_2.3x2mm_P0.5mm, symbol Logic_LevelTranslator:TXS0102DCU
- J503, J504: renamed from J?; footprint (none) -> Connector_PinSocket_2.54mm:PinSocket_1x10_P2.54mm_Vertical
- gave numbers to parts that had none: 2
- renumbered D501 to D502, D502 to D503, R501 to R502
Connections:
- net 3V3_CAN is gone; now on net GND: C502.1
- net CAN+ is gone; now on net MCU_CAN2H: D503.1 (A1), R502.1, U501.7 (CANH)
- net CAN- is gone; now on net MCU_CAN2L: D502.1 (A1), R502.2, U501.6 (CANL)
- net +3V3: now also C502.2, J503.2 (Pin_2), J504.2 (Pin_2), U502.3 (VCCA), U502.6 (OE)
- net +5V: now also U502.7 (VCCB)
- net GND: now also J501.4 (Pin_4), U502.2 (GND); no longer C502.2
- net Servo_RXD: now also J501.1 (Pin_1), U502.1 (B2)
- net Servo_TXD: now also J501.2 (Pin_2), U502.8 (B1)
- net Vdrive: now also J501.3 (Pin_3)
- net SHIELD_CAN2H: now reaches J504.3 (Pin_3)
- net SHIELD_CAN2H: now also J502.2
- net SHIELD_CAN2L: now reaches J504.4 (Pin_4)
- net SHIELD_CAN2L: now also J502.4
- net SHIELD_UART4_TX: now reaches J504.5 (Pin_5)
- net SHIELD_UART4_TX: now also U502.5 (A1)
- net SHIELD_UART4_RX: now reaches J504.6 (Pin_6)
- net SHIELD_UART4_RX: now also U502.4 (A2)
- net SHIELD_I2C1_SDA: now reaches J504.7 (Pin_7)
- net SHIELD_I2C1_SCL: now reaches J504.8 (Pin_8)
- net SHIELD_STAT_LED: now reaches D501.2 (A), J504.9 (Pin_9)
- net MCU_CAN2H: now reaches J503.3 (Pin_3)
- net MCU_CAN2L: now reaches J503.4 (Pin_4)
- net MCU_UART4_TX: now reaches J503.5 (Pin_5)
- net MCU_UART4_RX: now reaches J503.6 (Pin_6)
- net MCU_I2C1_SDA: now reaches J503.7 (Pin_7)
- net MCU_I2C1_SCL: now reaches J503.8 (Pin_8)
- net 57: now reaches J503.9 (Pin_9)
- net MCU_CAN1_RX renamed MCU_CAN2_RX
- net MCU_CAN1_TX renamed MCU_CAN2_TX
- no-connect marks 2 -> 4
Other:
- note added: "Servo Connector"
- note added: "Shield status LED"
- note removed: "Servo Connectors"
- moved on the sheet: D501, J503, J504, R501

Commit message: back from KL
Parts:
- added J505, J506: Conn_01x10, Connector_PinSocket_2.54mm:PinSocket_1x10_P2.54mm_Vertical, symbol Connector_Generic:Conn_01x10
Other:
- moved on the sheet: J502
