File: Misc.kicad_sch (KiCad schematic)
At the start: 20 parts, among them J501 Conn_01x04, J502 TE 338069-4, J503 Conn_01x10, J504 Conn_01x10, J505 Conn_01x10, J506 Conn_01x10, U501 SN65HVD232QDRQ1, U502 TXS0102DCU

Commit message: sIODGNIOSGDIONSHD
Parts:
- added J507, J508: Conn_02x05_Odd_Even, Connector_PinSocket_2.54mm:PinSocket_2x05_P2.54mm_Vertical, symbol Connector_Generic:Conn_02x05_Odd_Even
Other:
- moved on the sheet: J506

Commit message: asdbuioasdbgaseni
Connections:
- net +3V3: now also J505.1 (Pin_1), J507.1 (Pin_1)
- net +5V: now also J506.1 (Pin_1)
- net GND: now also J505.10 (Pin_10), J506.10 (Pin_10), J507.3 (Pin_3)
- net MCU_CAN1_TX: now reaches J507.2 (Pin_2)
- net MCU_CAN1_RX: now reaches J507.4 (Pin_4)
Other:
- moved on the sheet: J507, J508

Commit message: sdiognsidognsdb
Parts:
- added J509, J510: Conn_01x05, Connector_PinSocket_2.54mm:PinSocket_1x05_P2.54mm_Vertical, symbol Connector_Generic:Conn_01x05
Connections:
- net 57 is gone; now on net 35: J503.9 (Pin_9)
- net SHIELD_STAT_LED is gone; now on net 35: D501.2 (A), J504.9 (Pin_9)
- net +3V3: now also J505.2 (Pin_2), J506.2 (Pin_2), J508.1 (Pin_1); no longer J505.1 (Pin_1)
- net +5V: now also J505.1 (Pin_1)
- net GND: now also J508.3 (Pin_3)
- net MCU_CAN1_RX: now also J507.10 (Pin_10); no longer J507.4 (Pin_4)
- net MCU_CAN1_TX: now also J507.8 (Pin_8); no longer J507.2 (Pin_2)
- net 9: now reaches J507.5 (Pin_5)
- net 10: now reaches J507.6 (Pin_6)
- net 8: now reaches J507.7 (Pin_7)
- net 4: now reaches J507.9 (Pin_9)
- net SPI1_SCK: now reaches J506.7 (Pin_7)
- net SPI1_MISO: now reaches J506.8 (Pin_8)
- net SPI1_MOSI: now reaches J506.9 (Pin_9)
- net 35: now reaches J508.10 (Pin_10)
- net 35: now also J508.5 (Pin_5), J508.6 (Pin_6), J508.7 (Pin_7), J508.8 (Pin_8), J508.9 (Pin_9)
- net 2: now reaches J508.2 (Pin_2)
- net 3: now reaches J508.4 (Pin_4)
- new net 11: J507.4 (Pin_4)
- new net 16: J507.2 (Pin_2)
Other:
- note removed: "Shield status LED"
- moved on the sheet: J506, J507, J508

Commit message: sdgnseiogniosegn
Parts:
- removed J508: Conn_02x05_Odd_Even, Connector_PinSocket_2.54mm:PinSocket_2x05_P2.54mm_Vertical, symbol Connector_Generic:Conn_02x05_Odd_Even
Connections:
- net SPI1_SCK is gone; now on net MCU_I2C1_SDA: J506.7 (Pin_7)
- net 35: now also J503.10 (Pin_10), J504.10 (Pin_10); no longer J503.9 (Pin_9), J504.9 (Pin_9)
- net GND: now also J503.3 (Pin_3), J504.3 (Pin_3), J505.3 (Pin_3), J506.3 (Pin_3); no longer J503.10 (Pin_10), J504.10 (Pin_10), J505.10 (Pin_10), J506.10 (Pin_10)
- net MCU_CAN1_RX: now also J506.5 (Pin_5); no longer J507.10 (Pin_10)
- net MCU_CAN1_TX: now also J506.4 (Pin_4); no longer J507.8 (Pin_8)
- net MCU_CAN2H: now also J503.4 (Pin_4); no longer J503.3 (Pin_3)
- net MCU_CAN2L: now also J503.5 (Pin_5); no longer J503.4 (Pin_4)
- net MCU_I2C1_SCL: now also J506.6 (Pin_6); no longer J503.8 (Pin_8)
- net MCU_I2C1_SDA: no longer J503.7 (Pin_7)
- net MCU_UART4_RX: now also J503.7 (Pin_7); no longer J503.6 (Pin_6)
- net MCU_UART4_TX: now also J503.6 (Pin_6); no longer J503.5 (Pin_5)
- net SHIELD_CAN2H: now also J504.4 (Pin_4); no longer J504.3 (Pin_3)
- net SHIELD_CAN2L: now also J504.5 (Pin_5); no longer J504.4 (Pin_4)
- net SHIELD_I2C1_SCL: now also J505.6 (Pin_6); no longer J504.8 (Pin_8)
- net SHIELD_I2C1_SDA: now also J505.7 (Pin_7); no longer J504.7 (Pin_7)
- net SHIELD_UART4_RX: now also J504.7 (Pin_7); no longer J504.6 (Pin_6)
- net SHIELD_UART4_TX: now also J504.6 (Pin_6); no longer J504.5 (Pin_5)
- net SHIELD_CAN1_TX: now reaches J505.4 (Pin_4)
- net SHIELD_CAN1_RX: now reaches J505.5 (Pin_5)
- net SHIELD__SPI1_SCK: now reaches J505.8 (Pin_8)
- net SHIELD_SPI1_MISO: now reaches J505.9 (Pin_9)
- net SPI1_MISO renamed MCU__SPI1_SCK
- net SPI1_MOSI renamed MCU_SPI1_MISO
- new net MCU_SPI1_MOSI: J506.10 (Pin_10)
- new net SHIELD_SPI1_MOSI: J505.10 (Pin_10)
Other:
- moved on the sheet: J502, J503, J504, J505, J506, J507, J509, J510

Commit message: oenbioernb
Parts:
- removed H502, H504: MountingHole_Pad, MountingHole:MountingHole_3.2mm_M3_Pad_Via, symbol Mechanical:MountingHole_Pad
- removed J503: Conn_01x10, Connector_PinSocket_2.54mm:PinSocket_1x10_P2.54mm_Vertical, symbol Connector_Generic:Conn_01x10
- removed J507: Conn_02x05_Odd_Even, Connector_PinSocket_2.54mm:PinSocket_2x05_P2.54mm_Vertical, symbol Connector_Generic:Conn_02x05_Odd_Even
- added J?: Conn_01x13, symbol Connector_Generic:Conn_01x13
- renumbered H503 to H502
Connections:
- net +3V3: now also J?.5 (Pin_5); no longer J505.2 (Pin_2)
- net +5V: now also J?.4 (Pin_4); no longer J505.1 (Pin_1)
- net 35: now also J?.13 (Pin_13)
- net GND: now also J?.6 (Pin_6); no longer J505.3 (Pin_3)
- net MCU_CAN2H: now also J?.7 (Pin_7)
- net MCU_CAN2L: now also J?.8 (Pin_8)
- net MCU_UART4_RX: now also J?.10 (Pin_10)
- net MCU_UART4_TX: now also J?.9 (Pin_9)
- net MCU_USART3_TX: now reaches J504.8 (Pin_8)
- net MCU_USART3_TX: now also J?.11 (Pin_11)
- net MCU_USART3_RX: now reaches J504.9 (Pin_9)
- net MCU_USART3_RX: now also J?.12 (Pin_12)
- net 20: now reaches J510.1 (Pin_1)
- net 24: now reaches J510.2 (Pin_2)
- net 25: now reaches J510.3 (Pin_3)
- net 26: now reaches J510.4 (Pin_4)
- net 42: now reaches J510.5 (Pin_5)
- net SHIELD_CAN1_RX: no longer names the net of J505.5 (Pin_5)
- net SHIELD_CAN1_TX: no longer names the net of J505.4 (Pin_4)
- net SHIELD_I2C1_SCL: no longer names the net of J505.6 (Pin_6)
- net SHIELD_I2C1_SDA: no longer names the net of J505.7 (Pin_7)
- net SHIELD_SPI1_MISO: no longer names the net of J505.9 (Pin_9)
- net SHIELD_SPI1_MOSI: no longer names the net of J505.10 (Pin_10)
- net SHIELD__SPI1_SCK: no longer names the net of J505.8 (Pin_8)
- no-connect marks 4 -> 19
Other:
- note added: "Stacked socket header"
- moved on the sheet: C501, C502, C503, D501, D502, D503, H501, H502, J501, J502, J504, J505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

Commit message: sidbnb
Parts:
- removed J505, J506: Conn_01x10, Connector_PinSocket_2.54mm:PinSocket_1x10_P2.54mm_Vertical, symbol Connector_Generic:Conn_01x10
- removed J509, J510: Conn_01x05, Connector_PinSocket_2.54mm:PinSocket_1x05_P2.54mm_Vertical, symbol Connector_Generic:Conn_01x05
- removed J?: Conn_01x13, symbol Connector_Generic:Conn_01x13
- added J503: Conn_01x10, Connector_PinSocket_2.54mm:PinSocket_1x10_P2.54mm_Vertical, symbol Connector_Generic:Conn_01x10
- added J505, J506: Conn_01x13, Connector_PinSocket_2.54mm:PinSocket_1x13_P2.54mm_Vertical, symbol Connector_Generic:Conn_01x13
Connections:
- net +3V3: now also J503.2 (Pin_2), J506.2 (Pin_2)
- net +5V: now also J503.1 (Pin_1), J506.1 (Pin_1)
- net 35: now also J503.10 (Pin_10)
- net GND: now also J503.3 (Pin_3), J506.3 (Pin_3)
- net MCU_CAN1_RX: now also J505.5 (Pin_5)
- net MCU_CAN1_TX: now also J505.4 (Pin_4)
- net MCU_CAN2H: now also J503.4 (Pin_4)
- net MCU_CAN2L: now also J503.5 (Pin_5)
- net MCU_I2C1_SCL: now also J505.6 (Pin_6)
- net MCU_I2C1_SDA: now also J505.7 (Pin_7)
- net MCU_SPI1_MISO: now also J505.9 (Pin_9)
- net MCU_SPI1_MOSI: now also J505.10 (Pin_10)
- net MCU_UART4_RX: now also J503.7 (Pin_7)
- net MCU_UART4_TX: now also J503.6 (Pin_6)
- net MCU_USART3_RX: now also J503.9 (Pin_9)
- net MCU_USART3_TX: now also J503.8 (Pin_8)
- net MCU__SPI1_SCK: now also J505.8 (Pin_8)
- new net 10: J505.11 (Pin_11)
- new net 11: J505.12 (Pin_12)
- new net 16: J505.13 (Pin_13)
- no-connect marks 19 -> 17
Other:
- moved on the sheet: D501, J502, J504, R501

Commit message: sdighsidgh
Other:
- moved on the sheet: J503, J505, J506

Commit message: sdgnivvsdvinsv
Parts:
- removed J502: TE 338069-4, SnapEDA Library:TE_338069-4, symbol 338069-4:338069-4
- added J502: Conn_01x02, SnapEDA Library:JST_B2B-XH-A(LF)(SN), symbol Connector_Generic:Conn_01x02
Connections:
- net SHIELD_CAN2H: now also J502.2 (Pin_2)
- net SHIELD_CAN2L: now also J502.1 (Pin_1)
- net MCU__SPI1_SCK renamed MCU_SPI1_SCK
- no-connect marks 17 -> 15
Changed lines of the file:
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@@
   (no_connect (at 134.62 93.98))
   (no_connect (at 134.62 88.9))
-  (no_connect (at 44.45 99.06))
   (no_connect (at 187.96 49.53))
   (no_connect (at 187.96 52.07))
@@
   (no_connect (at 134.62 139.7))
   (no_connect (at 134.62 134.62))
-  (no_connect (at 44.45 93.98))
   (wire (pts (xy 181.61 81.28) (xy 190.5 81.28))
     (stroke (width 0) (type default) (color 0 0 0 0))
@@
   (label "CAN-" (at 190.5 46.99 0)
     (effects (font (size 0.4064 0.4064)) (justify left bottom))
+  )
+  (global_label "SHIELD_CAN2L" (shape input) (at 43.18 82.55 180) (fields_autoplaced)
+    (effects (font (size 1.27 1.27)) (justify right))
+    (property "Intersheet References" "${INTERSHEET_REFS}" (id 0) (at 27.3696 82.4706 0)
+      (effects (font (size 1.27 1.27)) (justify right) hide)
+    )
   )
   (global_label "Servo_RXD" (shape input) (at 62.23 34.29 180) (fields_autoplaced)
@@
     )
   )
-  (global_label "SHIELD_CAN2L" (shape input) (at 44.45 91.44 180) (fields_autoplaced)
-    (effects (font (size 1.27 1.27)) (justify right))
-    (property "Intersheet References" "${INTERSHEET_REFS}" (id 0) (at 28.6396 91.3606 0)
-      (effects (font (size 1.27 1.27)) (justify right) hide)
-    )
-  )
   (global_label "MCU_UART4_TX" (shape input) (at 95.25 153.67 180) (fields_autoplaced)
     (effects (font (size 1.27 1.27)) (justify right))
@@
     )
   )
-  (global_label "SHIELD_CAN2H" (shape input) (at 44.45 96.52 180) (fields_autoplaced)
-    (effects (font (size 1.27 1.27)) (justify right))
-    (property "Intersheet References" "${INTERSHEET_REFS}" (id 0) (at 28.3372 96.4406 0)
-      (effects (font (size 1.27 1.27)) (justify right) hide)
-    )
-  )
   (global_label "Servo_TXD" (shape input) (at 62.23 36.83 180) (fields_autoplaced)
     (effects (font (size 1.27 1.27)) (justify right))
@@
     )
   )
+  (global_label "SHIELD_CAN2H" (shape input) (at 43.18 85.09 180) (fields_autoplaced)
+    (effects (font (size 1.27 1.27)) (justify right))
+    (property "Intersheet References" "${INTERSHEET_REFS}" (id 0) (at 27.0672 85.0106 0)
+      (effects (font (size 1.27 1.27)) (justify right) hide)
+    )
+  )
   (global_label "MCU_SPI1_MOSI" (shape input) (at 134.62 157.48 180) (fields_autoplaced)
     (effects (font (size 1.27 1.27)) (justify right))
@@
     )
   )
-  (global_label "MCU__SPI1_SCK" (shape input) (at 134.62 152.4 180) (fields_autoplaced)
-    (effects (font (size 1.27 1.27)) (justify right))
-    (property "Intersheet References" "${INTERSHEET_REFS}" (id 0) (at 117.2977 152.3206 0)
+  (global_label "MCU_SPI1_SCK" (shape input) (at 134.62 152.4 180) (fields_autoplaced)
+    (effects (font (size 1.27 1.27)) (justify right))
+    (property "Intersheet References" "${INTERSHEET_REFS}" (id 0) (at 118.2653 152.3206 0)
       (effects (font (size 1.27 1.27)) (justify right) hide)
     )
@@
     (pin "2")
   )
-  (symbol (lib_id "338069-4:338069-4") (at 52.07 93.98 180) (unit 1)
-    (in_bom yes) (on_board yes)
-    (property "Reference" "J502" (id 0) (at 57.15 101.6 90)
-      (effects (font (size 1.27 1.27)) (justify right))
-    )
-    (property "Value" "TE 338069-4" (id 1) (at 59.69 101.6 90)
-      (effects (font (size 1.27 1.27)) (justify right))
-    )
-    (property "Footprint" "SnapEDA Library:TE_338069-4" (id 2) (at 52.07 93.98 0)
-      (effects (font (size 1.27 1.27)) (justify left bottom) hide)
-    )
-    (property "Datasheet" "" (id 3) (at 52.07 93.98 0)
-      (effects (font (size 1.27 1.27)) (justify left bottom) hide)
-    )
-    (property "STANDARD" "Manufacturer Recommendation" (id 4) (at 52.07 93.98 0)
-      (effects (font (size 1.27 1.27)) (justify left bottom) hide)
-    )
-    (property "MANUFACTURER" "TE Connectivity AMP Connectors" (id 5) (at 52.07 93.98 0)
-      (effects (font (size 1.27 1.27)) (justify left bottom) hide)
-    )
-    (property "SERIES" "Micro-MaTch" (id 6) (at 52.07 93.98 0)
-      (effects (font (size 1.27 1.27)) (justify left bottom) hide)
-    )
-    (property "POSITIONS" "14" (id 7) (at 52.07 93.98 0)
-      (effects (font (size 1.27 1.27)) (justify left bottom) hide)
-    )
-    (property "PITCH" "2.54mm" (id 8) (at 52.07 93.98 0)
-      (effects (font (size 1.27 1.27)) (justify left bottom) hide)
-    )
-    (property "VOLTAGE" "100VDC" (id 9) (at 52.07 93.98 0)
-      (effects (font (size 1.27 1.27)) (justify left bottom) hide)
-    )
-    (property "PARTREV" "H4" (id 10) (at 52.07 93.98 0)
-      (effects (font (size 1.27 1.27)) (justify left bottom) hide)
-    )
-    (pin "1")
-    (pin "2")
-    (pin "3")
-    (pin "4")
-  )
   (symbol (lib_id "Connector_Generic:Conn_01x10") (at 101.6 95.25 0) (unit 1)
     (in_bom yes) (on_board yes)
@@
     (pin "1")
   )
+  (symbol (lib_id "Connector_Generic:Conn_01x02") (at 48.26 82.55 0) (unit 1)
+    (in_bom yes) (on_board yes) (fields_autoplaced)
+    (property "Reference" "J502" (id 0) (at 50.8 82.5499 0)
+      (effects (font (size 1.27 1.27)) (justify left))
+    )
+    (property "Value" "Conn_01x02" (id 1) (at 50.8 85.0899 0)
+      (effects (font (size 1.27 1.27)) (justify left))
+    )
+    (property "Footprint" "SnapEDA Library:JST_B2B-XH-A(LF)(SN)" (id 2) (at 48.26 82.55 0)
+      (effects (font (size 1.27 1.27)) hide)
+    )
+    (property "Datasheet" "~" (id 3) (at 48.26 82.55 0)
+      (effects (font (size 1.27 1.27)) hide)
+    )
+    (pin "1")
+    (pin "2")
+  )
   (symbol (lib_id "BluePhil-rescue:+3.3V-power") (at 157.48 29.21 0) (unit 1)
