File: MCU.kicad_sch (KiCad schematic)
At the start: 37 parts, among them J301 SWD, J302 USB_C_Receptacle_USB2.0, SW301 SW_SPDT, U301 STM32F405RGT6, U302 USBLC6-2SC6, Y301 16MHz

Commit message: final commit before holiday
Parts:
- removed D306: RCLAMP0521P-N, Diode_SMD:D_0402_1005Metric, symbol Device:D_TVS
- removed J302: USB_C_Receptacle_USB2.0, Connector_USB:USB_C_Receptacle_XKB_U262-16XN-4BVC11, symbol Connector:USB_C_Receptacle_USB2.0
- removed R312, R313: 2k2, Resistor_SMD:R_0402_1005Metric, symbol Device:R_Small
- added D307: RCLAMP0521P-N, Diode_SMD:D_0402_1005Metric, symbol Device:D_TVS
- added J303: USB4520-03-0-A_REVA, SnapEDA Library:GCT_USB4520-03-0-A_REVA, symbol USB4520-03-0-A_REVA:USB4520-03-0-A_REVA
- added R314, R315: 5k1, Resistor_SMD:R_0402_1005Metric, symbol Device:R_Small
Connections:
- net 56 is gone; now on net IMU_INTERRUPT: U301.56 (PB4)
- net CONN_USB_D+: now also J303.A6 (DP1), J303.B6 (DP2)
- net CONN_USB_D-: now also J303.A7 (DN1), J303.B7 (DN2)
- net GND: now also D307.2 (A2), J303.A1_B12 (GND_A), J303.B1_A12 (GND_B), J303.S1 (SHELL_GND), J303.S2 (SHELL_GND), J303.S3 (SHELL_GND), J303.S4 (SHELL_GND), R314.1, R315.2
- net IMU_INTERRUPT: no longer U301.27 (PB1)
- net VBUS: now also D307.1 (A1), J303.A4_B9 (VBUS_A), J303.B4_A9 (VBUS_B)
- net 33 renamed MCU_CAN2_RX
- net 34 renamed MCU_CAN2_TX
- net MCU_RXD renamed MCU_UART4_RX
- net MCU_TXD renamed MCU_UART4_TX
- new net: J303.B5 (CC2), R315.1
- new net: J303.A5 (CC1), R314.2
- new net 27: U301.27 (PB1)
- no-connect marks 7 -> 6
Other:
- moved on the sheet: C312, D302, D303, D304, D305, J301, R304, R309, R310, R311, U302

Commit message: sdgihisodgn
Parts:
- added R301, R307: 2k2, Resistor_SMD:R_0402_1005Metric, symbol Device:R_Small
- renumbered D307 to D306, J303 to J302, R301 to R302, R302 to R303, R303 to R306, R304 to R308, R305 to R309, R306 to R310, R307 to R311, R308 to R312, R314 to R313, R309 to R314, R310 to R315, R311 to R316, R315 to R317
Connections:
- net +3V3: now also R301.1, R307.1
- net 40 renamed MCU_I2C3_SDA
- net MCU_I2C3_SDA: now also R301.2
- net 41 renamed MCU_I2C3_SCL
- net MCU_I2C3_SCL: now also R307.2
Other:
- note added: "JTAG/SWD"
- note added: "USB C Receptacle and ESD Protection"
- note removed: "SWD"
- note removed: "USB C"

Commit message: sIODGNIOSGDIONSHD
Parts:
- removed J302: USB4520-03-0-A_REVA, SnapEDA Library:GCT_USB4520-03-0-A_REVA, symbol USB4520-03-0-A_REVA:USB4520-03-0-A_REVA
- removed R313, R317: 5k1, Resistor_SMD:R_0402_1005Metric, symbol Device:R_Small
- added J302: USB4085-GF-A_REVA4, SnapEDA Library:GCT_USB4085-GF-A_REVA4, symbol USB4085-GF-A:USB4085-GF-A_REVA4
- added R304, R305: 5k1, Resistor_SMD:R_0402_1005Metric, symbol Device:R_Small
Connections:
- net CONN_USB_D+: now also J302.A6 (DP1), J302.B6 (DP2)
- net CONN_USB_D-: now also J302.A7 (DN1), J302.B7 (DN2)
- net GND: now also J302.A1 (GND), J302.A12 (GND), J302.B1 (GND), J302.B12 (GND), J302.S1 (SHELL), J302.S2 (SHELL), J302.S3 (SHELL), J302.S4 (SHELL), R304.1, R305.1
- net VBUS: now also J302.A4 (VBUS), J302.A9 (VBUS), J302.B4 (VBUS), J302.B9 (VBUS)
- new net: J302.B5 (CC2), R305.2
- new net: J302.A5 (CC1), R304.2

Commit message: sdiognsidognsdb
Connections:
- net 27 is gone; now on net IMU_INTERRUPT: U301.27 (PB1)
- net IMU_INTERRUPT: no longer U301.56 (PB4)
- net 21 renamed SPI1_SCK
- net 22 renamed SPI1_MISO
- net 23 renamed SPI1_MOSI
- net 35 renamed SHIELD_STAT_LED
- new net 56: U301.56 (PB4)
Other:
- moved on the sheet: R307

Commit message: sdgnseiogniosegn
Connections:
- net SPI1_MISO renamed MCU_SPI1_MISO
- net SPI1_MOSI renamed MCU_SPI1_MOSI
- net SPI1_SCK renamed MCU_SPI1_SCK
Changed lines of the file:
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@@
     )
   )
-  (global_label "SPI1_MISO" (shape input) (at 101.6 93.98 0) (fields_autoplaced)
-    (effects (font (size 1.27 1.27)) (justify left))
-    (property "Intersheet References" "${INTERSHEET_REFS}" (id 0) (at 113.7818 94.0594 0)
+  (global_label "MCU_SPI1_MISO" (shape input) (at 101.6 93.98 0) (fields_autoplaced)
+    (effects (font (size 1.27 1.27)) (justify left))
+    (property "Intersheet References" "${INTERSHEET_REFS}" (id 0) (at 118.8013 93.9006 0)
       (effects (font (size 1.27 1.27)) (justify left) hide)
     )
@@
     )
   )
-  (global_label "SPI1_SCK" (shape input) (at 101.6 91.44 0) (fields_autoplaced)
-    (effects (font (size 1.27 1.27)) (justify left))
-    (property "Intersheet References" "${INTERSHEET_REFS}" (id 0) (at 112.9352 91.5194 0)
+  (global_label "MCU_SPI1_SCK" (shape input) (at 101.6 91.44 0) (fields_autoplaced)
+    (effects (font (size 1.27 1.27)) (justify left))
+    (property "Intersheet References" "${INTERSHEET_REFS}" (id 0) (at 117.9547 91.3606 0)
       (effects (font (size 1.27 1.27)) (justify left) hide)
     )
@@
     )
   )
-  (global_label "SPI1_MOSI" (shape input) (at 101.6 96.52 0) (fields_autoplaced)
-    (effects (font (size 1.27 1.27)) (justify left))
-    (property "Intersheet References" "${INTERSHEET_REFS}" (id 0) (at 113.7818 96.5994 0)
-      (effects (font (size 1.27 1.27)) (justify left) hide)
-    )
+  (global_label "MCU_SPI1_MOSI" (shape input) (at 101.6 96.52 0) (fields_autoplaced)
+    (effects (font (size 1.27 1.27)) (justify left))
+    (property "Intersheet References" "${INTERSHEET_REFS}" (id 0) (at 118.8013 96.4406 0)
+      (effects (font (size 1.27 1.27)) (justify left) hide)
+    )

Commit message: oenbioernb
Connections:
- net 51 renamed MCU_USART3_TX
- net 52 renamed MCU_USART3_RX
Changed lines of the file:
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@@
+    )
+  )
+  (global_label "MCU_USART3_TX" (shape output) (at 66.04 147.32 180) (fields_autoplaced)
+    (effects (font (size 1.27 1.27)) (justify right))
+    (property "Intersheet References" "${INTERSHEET_REFS}" (id 0) (at 48.4758 147.2406 0)
+      (effects (font (size 1.27 1.27)) (justify right) hide)
     )
   )
@@
     (effects (font (size 1.27 1.27)) (justify right))
     (property "Intersheet References" "${INTERSHEET_REFS}" (id 0) (at 61.2968 129.4606 0)
-      (effects (font (size 1.27 1.27)) (justify right) hide)
-    )
-  )
-  (global_label "51" (shape input) (at 66.04 147.32 180) (fields_autoplaced)
-    (effects (font (size 1.27 1.27)) (justify right))
-    (property "Intersheet References" "${INTERSHEET_REFS}" (id 0) (at 61.2968 147.2406 0)
       (effects (font (size 1.27 1.27)) (justify right) hide)
     )
@@
     )
   )
-  (global_label "MCU_SPI1_SCK" (shape input) (at 101.6 91.44 0) (fields_autoplaced)
+  (global_label "MCU_SPI1_SCK" (shape output) (at 101.6 91.44 0) (fields_autoplaced)
     (effects (font (size 1.27 1.27)) (justify left))
     (property "Intersheet References" "${INTERSHEET_REFS}" (id 0) (at 117.9547 91.3606 0)
@@
     )
   )
-  (global_label "MCU_UART4_TX" (shape input) (at 101.6 78.74 0) (fields_autoplaced)
+  (global_label "MCU_UART4_TX" (shape output) (at 101.6 78.74 0) (fields_autoplaced)
     (effects (font (size 1.27 1.27)) (justify left))
     (property "Intersheet References" "${INTERSHEET_REFS}" (id 0) (at 117.9547 78.6606 0)
@@
     )
   )
-  (global_label "52" (shape input) (at 66.04 149.86 180) (fields_autoplaced)
+  (global_label "MCU_USART3_RX" (shape input) (at 66.04 149.86 180) (fields_autoplaced)
     (effects (font (size 1.27 1.27)) (justify right))
-    (property "Intersheet References" "${INTERSHEET_REFS}" (id 0) (at 61.2968 149.7806 0)
+    (property "Intersheet References" "${INTERSHEET_REFS}" (id 0) (at 48.1734 149.7806 0)
       (effects (font (size 1.27 1.27)) (justify right) hide)
     )
@@
     )
   )
-  (global_label "MCU_SPI1_MOSI" (shape input) (at 101.6 96.52 0) (fields_autoplaced)
+  (global_label "MCU_SPI1_MOSI" (shape output) (at 101.6 96.52 0) (fields_autoplaced)
     (effects (font (size 1.27 1.27)) (justify left))
     (property "Intersheet References" "${INTERSHEET_REFS}" (id 0) (at 118.8013 96.4406 0)
@@
     )
   )
-  (global_label "SHIELD_STAT_LED" (shape input) (at 123.19 162.56 0) (fields_autoplaced)
+  (global_label "SHIELD_STAT_LED" (shape output) (at 123.19 162.56 0) (fields_autoplaced)
     (effects (font (size 1.27 1.27)) (justify left))
     (property "Intersheet References" "${INTERSHEET_REFS}" (id 0) (at 141.7218 162.4806 0)

Commit message: sdighsidgh
Parts:
- removed J302: USB4085-GF-A_REVA4, SnapEDA Library:GCT_USB4085-GF-A_REVA4, symbol USB4085-GF-A:USB4085-GF-A_REVA4
- added J302: USB4110-GF-A_REVB, SnapEDA Library:GCT_USB4110-GF-A_REVB, symbol USB4110:USB4110-GF-A_REVB
Connections:
- net CONN_USB_D+: now also J302.A6 (DP1), J302.B6 (DP2)
- net CONN_USB_D-: now also J302.A7 (DN1), J302.B7 (DN2)
- net GND: now also R305.2, J302.A1/B12 (GND), J302.B1/A12 (GND), J302.S1 (GND), J302.S2 (GND), J302.S3 (GND), J302.S4 (GND); no longer R305.1
- net VBUS: now also J302.A4/B9 (VBUS), J302.B4/A9 (VBUS)
- net at R304.2: now also J302.A5 (CC1)
- new net: J302.B5 (CC2), R305.1
