File: Sensors_with_jumper_bridge.kicad_sch (KiCad schematic)
At the start: 7 parts, among them J401 BM04B-SURS-TFLFSN, U401 ICM-42670-P

Commit message: incorporated rework into official design
Parts:
- added JP401, JP402: (no value), symbol Jumper:SolderJumper_3_Bridged12
- C401: value 10n -> (none); footprint Capacitor_SMD:C_0402_1005Metric -> (none)
- C402: value 0.1u -> (none); footprint Capacitor_SMD:C_0402_1005Metric -> (none)
- C403: value 2u2 -> (none); footprint Capacitor_SMD:C_0402_1005Metric -> (none)
- J401: value BM04B-SURS-TFLFSN -> (none); footprint SnapEDA Library:JST_BM04B-SURS-TF(LF)(SN) -> (none)
- R401, R402: value 0R -> (none); footprint Resistor_SMD:R_0402_1005Metric -> (none)
- U401: value ICM-42670-P -> (none); footprint SnapEDA Library:IC_ICM-42670-P -> (none)
Connections:
- net +3V3: now also JP401.3 (B), JP402.1 (A); no longer J401.1
- net GND: now also JP401.1 (A), JP402.3 (B); no longer J401.4
- new net: J401.4, JP402.2 (C)
- new net: J401.1, JP401.2 (C)
